File: Block Diagram.kicad_sch (KiCad schematic)
At the start: 0 parts

Commit message: Progress on Block Diagram
Other:
- note added: "+12V"
- note added: "+5v"
- note removed: "+??V"
- note removed: "+A3V3"
