File: Drives.kicad_sch (KiCad schematic)
At the start: 0 parts

Commit message: Libaries added
Parts:
- added C18, C28: 22u, symbol Device:C_Small
- added C23, C24, C25, C26, C30, C31, C32, C33: 22n, symbol Device:C_Small
- added C27: 100n, Capacitor_SMD:C_0402_1005Metric, symbol Device:C
- added C29, C9: 100n, symbol Device:C_Small
- added D5: LED Green, LED_SMD:LED_0603_1608Metric, symbol Device:LED
- added IC1, IC2: AP62800SJ-7, AP62800SJ7, symbol AP62800SJ-7:AP62800SJ-7
- added J10: Conn_01x03_Pin, symbol Connector:Conn_01x03_Pin
- added J11: Bus_M.2_Socket_M, CM5IO:M.2 M Key socket, symbol CM5IO:Bus_M.2_Socket_M
- added J3, J4: Conn_02x03_Odd_Even, symbol Connector_Generic:Conn_02x03_Odd_Even
- added L1, L2: 2u, symbol Device:L
- added M1, M10, M15, M20: M.2 Screw, symbol CM5IO:M.2_Screw
- added M11, M12, M13, M14, M16, M17, M18, M19, M2, M3, M4, M5, M6, M7, M8, M9: M.2 Solder Nut, symbol CM5IO:SolderNut
- added Q1: Q_PMOS, symbol Device:Q_PMOS
- added R11, R15: 30.1k, symbol Device:R
- added R12, R8: R, symbol Device:R
- added R13, R14: 100K 1%, Resistor_SMD:R_0402_1005Metric, symbol Device:R
- added R16, R9: 137k, symbol Device:R
- added R17: 1k, Resistor_SMD:R_0402_1005Metric, symbol Device:R
- added TP1: TestPoint, TestPoint:TestPoint_Pad_2.0x2.0mm, symbol Connector:TestPoint
- added U7: ASEK-32.768KHZ-L-R-T, Crystal:Crystal_SMD_3225-4Pin_3.2x2.5mm, symbol CM5IO:ASEK-32.768KHZ-L-R-T
Connections:
- new net: J10.1 (Pin_1), Q1.G
- new net: D5.1 (K), R17.1, TP1.1
- new net: J11.10 (DAS/~{DSS}/~{LED1}), R17.2
- new net: J11.68 (SUSCLK), U7.3 (Out)
- new net: IC1.12 (FB), R11.2, R9.2
- new net: IC2.12 (FB), R15.2, R16.2
- new net: IC2.6 (PG), R12.2
- new net: C29.1, IC2.7 (BST)
- new net: C29.2, IC2.8 (SW), L2.1
- new net: IC1.6 (PG), R8.2
- new net: C9.2, IC1.8 (SW), L1.1
- new net: C9.1, IC1.7 (BST)
- new net +12v: Q1.S
- new net +5v: C18.1, C28.1, IC1.2 (VIN), IC1.3 (EN), IC1.4 (MODE), IC1.9 (VCC), IC2.2 (VIN), IC2.3 (EN), IC2.4 (MODE), IC2.9 (VCC), J10.2 (Pin_2), J3.3 (Pin_3), J3.4 (Pin_4), J4.3 (Pin_3), J4.4 (Pin_4), R12.1, R13.1, R14.1, R8.1
- new net GND: C18.2, C23.2, C24.2, C25.2, C26.2, C27.2, C28.2, C30.2, C31.2, C32.2, C33.2, IC1.1 (PGND), IC1.11 (GND), IC1.5 (FSEL), IC2.1 (PGND), IC2.11 (GND), IC2.5 (FSEL), J11.1 (GND), J11.15 (GND), J11.21 (GND), J11.27 (GND), J11.3 (GND), J11.33 (GND), J11.39 (GND), J11.45 (GND), J11.51 (GND), J11.57 (GND), J11.71 (GND), J11.73 (GND), J11.75 (GND), J11.9 (GND), J11.M1 (GND2230), J11.M2 (GND2242), J11.M3 (GND2260), J11.M4 (GND2280), J11.S1, J11.S2, J3.1 (Pin_1), J3.2 (Pin_2), J4.1 (Pin_1), J4.2 (Pin_2), R11.1, R13.2, R14.2, R15.1, U7.2 (GND)
- new net M2_3v3: C27.1, D5.2 (A), J11.12 (3.3V), J11.14 (3.3V), J11.16 (3.3V), J11.18 (3.3V), J11.2 (3.3V), J11.4 (3.3V), J11.70 (3.3V), J11.72 (3.3V), J11.74 (3.3V), U7.1 (EN), U7.4 (VDD)
- new net M2_3v3 (1): C30.1, C31.1, C32.1, C33.1, L2.2, R16.1
- new net M2_3v3 (2): C23.1, C24.1, C25.1, C26.1, L1.2, R9.1
- new net SATA +12v: J3.5 (Pin_5), J3.6 (Pin_6), J4.5 (Pin_5), J4.6 (Pin_6), Q1.D
- no-connect marks 0 -> 17
Other:
- note added: "Activity LED"

Commit message: Voltage calcs
Parts:
- removed J10: Conn_01x03_Pin, symbol Connector:Conn_01x03_Pin
- removed J3, J4: Conn_02x03_Odd_Even, symbol Connector_Generic:Conn_02x03_Odd_Even
- removed Q1: Q_PMOS, symbol Device:Q_PMOS
- added C21, C22, C23, C24, C25, C26, C29, C30, C31, C32, C33, C34, C35, C36, C37, C38, C39, C40, C51, C52, C53, C54, C55, C56, C57, C58, C59, C60: 100nF, Capacitor_SMD:C_0402_1005Metric, symbol Device:C
- added C62: 22n, symbol Device:C_Small
- added R13, R16, R20, R22: 1K, Resistor_SMD:R_0402_1005Metric, symbol Device:R
- added R19, R21, R23, R24, R26: 10K, Resistor_SMD:R_0402_1005Metric, symbol Device:R
- added R25, R27: 12.1K, Resistor_SMD:R_0402_1005Metric, symbol Device:R
- added R29: 10k, symbol Device:R
- added U7: ASM1184, Package_DFN_QFN:QFN-64-1EP_9x9mm_P0.5mm_EP5.2x5.2mm, symbol ASM1184:ASM1184
- added U9: TMP102xxDRL, Package_TO_SOT_SMD:SOT-563, symbol Sensor_Temperature:TMP102xxDRL
- renumbered C28 to C27, C18 to C28, C29 to C41, C9 to C42, C30 to C43, C23 to C44, C31 to C45, C24 to C46, C32 to C47, C25 to C48, C33 to C49, C26 to C50, C27 to C61, IC2 to IC1, IC1 to IC2, J11 to J13, L2 to L1, L1 to L2, M6 to M1, M1 to M10, M7 to M2, M8 to M3, M9 to M4, M10 to M5, M5 to M6, M4 to M7, M3 to M8, M2 to M9, R8 to R10, R13 to R11, R14 to R12, R15 to R14, R11 to R15, R16 to R17, R9 to R18, R17 to R28, R12 to R9, TP1 to TP3, U7 to U8
Connections:
- net GND: now also C21.2, C22.2, C23.2, C24.2, C25.2, C26.2, C29.2, C30.2, C31.2, C32.2, C33.2, C34.2, C35.2, C36.2, C37.2, C38.2, C39.2, C40.2, C62.2, R13.2, R16.2, R20.2, R22.2, R25.2, R27.2, U7.53 (GND), U7.65 (GND), U9.2 (GND), U9.4 (ADD0)
- net PCIE_CLK_N: now also U7.47 (REFCLKN_IN)
- net PCIE_CLK_P: now also U7.46 (REFCLKP_IN)
- net PCIE_RX_N: now also U7.52 (RXN_IN)
- net PCIE_RX_P: now also U7.51 (RXP_IN)
- net PCIE_TX_N: now also C60.1
- net PCIE_TX_P: now also C59.1
- new net: R25.1, U7.16 (REXT1)
- new net: C58.2, U7.58 (TXN_4)
- new net: R19.2, U7.31 (GPIO_1)
- new net: R27.1, U7.49 (REXT2)
- new net: R23.2, U7.36 (GPIO_7)
- new net: C51.2, U7.11 (TXP_1)
- new net: C52.2, U7.12 (TXN_1)
- new net: C53.2, U7.22 (TXP_2)
- new net: C54.2, U7.23 (TXN_2)
- new net: R21.2, U7.30 (GPIO_5)
- new net: R22.1, U7.33 (TEST_EN)
- new net: R24.2, U7.34 (GPIO_3)
- new net: R20.1, U7.35 (GPIO_6)
- new net: C55.2, U7.39 (TXP_3)
- new net: R26.2, U7.4 (GPIO_0)
- new net: C56.2, U7.40 (TXN_3)
- new net: R16.1, U7.5 (GPIO_2)
- new net: C59.2, U7.54 (TXP_IN)
- new net: C60.2, U7.55 (TXN_IN)
- new net: C57.2, U7.57 (TXP_4)
- new net: R13.1, U7.8 (GPIO_4)
- new net: C62.1, R29.2, U9.5 (V+)
- new net +1V2: C21.1, C22.1, C24.1, C25.1, C29.1, C30.1, C32.1, C33.1, C35.1, C36.1, C38.1, C39.1, U7.15 (1V2), U7.17 (1V2), U7.20 (1V2), U7.26 (1V2), U7.29 (1V2), U7.37 (1V2), U7.43 (1V2), U7.48 (1V2), U7.50 (1V2), U7.61 (1V2), U7.64 (1V2), U7.9 (1V2)
- new net +3.3VA: C23.1, C26.1, C31.1, C34.1, C37.1, C40.1, R19.1, R21.1, R23.1, R24.1, R26.1, U7.1 (3V_AUX), U7.10 (3V3), U7.21 (3V3), U7.32 (3V3), U7.38 (3V3), U7.56 (3V3)
- new net +3V3: R29.1
- new net PCIe_CLK_N_1: U7.19 (REFCLKN_1)
- new net PCIe_CLK_N_2: U7.28 (REFCLKN_2)
- new net PCIe_CLK_N_3: U7.45 (REFCLKN_3)
- new net PCIe_CLK_N_4: U7.63 (REFCLKN_4)
- new net PCIe_CLK_P_1: U7.18 (REFCLKP_1)
- new net PCIe_CLK_P_2: U7.27 (REFCLKP_2)
- new net PCIe_CLK_P_3: U7.44 (REFCLKP_3)
- new net PCIe_CLK_P_4: U7.62 (REFCLKP_4)
- new net PCIe_RST: U7.3 (RES_IN)
- new net PCIe_RST_M2: U7.2 (RES_OUT)
- new net PCIe_RX_N_1: U7.14 (RXN_1)
- new net PCIe_RX_N_2: U7.25 (RXN_2)
- new net PCIe_RX_N_3: U7.42 (RXN_3)
- new net PCIe_RX_N_4: U7.60 (RXN_4)
- new net PCIe_RX_P_1: U7.13 (RXP_1)
- new net PCIe_RX_P_2: U7.24 (RXP_2)
- new net PCIe_RX_P_3: U7.41 (RXP_3)
- new net PCIe_RX_P_4: U7.59 (RXP_4)
- new net PCIe_TX_N_1: C52.1
- new net PCIe_TX_N_2: C54.1
- new net PCIe_TX_N_3: C56.1
- new net PCIe_TX_N_4: C58.1
- new net PCIe_TX_P_1: C51.1
- new net PCIe_TX_P_2: C53.1
- new net PCIe_TX_P_3: C55.1
- new net PCIe_TX_P_4: C57.1
- new net SCL0: U9.1 (SCL)
- new net SDA0: U9.6 (SDA)
