File: Electronics/Block Diagram.kicad_sch (KiCad schematic)
At the start: 0 parts

Commit message: Footprints Selected
Other:
- note added: "+5V"
- note removed: "+5v"
Changed lines of the file:
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@@
 		)
 	)
-	(text "+5v"
+	(text "+5V"
 		(exclude_from_sim no)
 		(at 347.726 106.68 0)
@@
 		)
 	)
-	(text "+5v"
+	(text "+5V"
 		(exclude_from_sim no)
 		(at 138.176 88.646 0)
@@
 		)
 	)
-	(text "+5v"
+	(text "+5V"
 		(exclude_from_sim no)
 		(at 114.046 88.646 0)

Commit message: Footprints selected, Hiracicle connections created, Pcb next
Changed lines of the file:
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@@
+		)
+	)
+	(text_box "Page 5"
+		(exclude_from_sim no)
+		(at 156.21 78.105 0)
+		(size 24.765 5.08)
+		(margins 1.7144 1.7144 1.7144 1.7144)
+		(stroke
+			(width -0.0001)
+			(type default)
+		)
+		(fill
+			(type none)
+		)
+		(effects
+			(font
+				(face "Times New Roman")
+				(size 2.286 2.286)
+				(thickness 0.4572)
+				(bold yes)
+				(color 0 0 0 1)
+			)
+			(justify left top)
+			(href "#5")
 		)
 	)
@@
 				(color 0 0 0 1)
 			)
-		)
-	)
-	(text_box "Page 8"
-		(exclude_from_sim no)
-		(at 302.006 97.028 0)
-		(size 17.78 5.08)
-		(margins 1.7144 1.7144 1.7144 1.7144)
-		(stroke
-			(width -0.0001)
-			(type solid)
-		)
-		(fill
-			(type none)
-		)
-		(effects
-			(font
-				(face "Times New Roman")
-				(size 2.286 2.286)
-				(thickness 0.4572)
-				(bold yes)
-				(color 0 0 0 1)
-			)
-			(justify left top)
-			(href "#8")
 		)
 	)
@@
 		)
 	)
+	(text_box "Page 8"
+		(exclude_from_sim no)
+		(at 300.99 85.09 0)
+		(size 17.78 5.08)
+		(margins 1.7144 1.7144 1.7144 1.7144)
+		(stroke
+			(width -0.0001)
+			(type solid)
+		)
+		(fill
+			(type none)
+		)
+		(effects
+			(font
+				(face "Times New Roman")
+				(size 2.286 2.286)
+				(thickness 0.4572)
+				(bold yes)
+				(color 0 0 0 1)
+			)
+			(justify left top)
+			(href "#8")
+		)
+	)
 	(text_box "DSI"
 		(exclude_from_sim no)
@@
 		)
 	)
+	(text_box "Page 4"
+		(exclude_from_sim no)
+		(at 156.21 73.66 0)
+		(size 24.765 5.08)
+		(margins 1.7144 1.7144 1.7144 1.7144)
+		(stroke
+			(width -0.0001)
+			(type default)
+		)
+		(fill
+			(type none)
+		)
+		(effects
+			(font
+				(face "Times New Roman")
+				(size 2.286 2.286)
+				(thickness 0.4572)
+				(bold yes)
+				(color 0 0 0 1)
+			)
+			(justify left top)
+		)
+	)
 	(text_box "\nL\n\n\nN\n\n\n\n\n\n"
 		(exclude_from_sim no)
@@
 		)
 	)
-	(text_box "88 ~ 132VAC / 176 ~ 264VAC selected by switch"
+	(text_box "88 gnd 132VAC / 176 gnd 264VAC selected by switch"
 		(exclude_from_sim no)
 		(at 370.84 182.88 0)
@@
 		)
 	)
+	(text_box "Page 9"
+		(exclude_from_sim no)
+		(at 300.99 88.9 0)
+		(size 17.78 5.08)
+		(margins 1.7144 1.7144 1.7144 1.7144)
+		(stroke
+			(width -0.0001)
+			(type solid)
+		)
+		(fill
+			(type none)
+		)
+		(effects
+			(font
+				(face "Times New Roman")
+				(size 2.286 2.286)
+				(thickness 0.4572)
+				(bold yes)
+				(color 0 0 0 1)
+			)
+			(justify left top)
+			(href "#9")
+		)
+	)
 	(text_box "USB 3.0"
 		(exclude_from_sim no)
@@
 		)
 	)
+	(text_box "Page 11"
+		(exclude_from_sim no)
+		(at 300.99 96.52 0)
+		(size 17.78 5.08)
+		(margins 1.7144 1.7144 1.7144 1.7144)
+		(stroke
+			(width -0.0001)
+			(type solid)
+		)
+		(fill
+			(type none)
+		)
+		(effects
+			(font
+				(face "Times New Roman")
+				(size 2.286 2.286)
+				(thickness 0.4572)
+				(bold yes)
+				(color 0 0 0 1)
+			)
+			(justify left top)
+			(href "#11")
+		)
+	)
+	(text_box "Page 10"
+		(exclude_from_sim no)
+		(at 300.99 92.71 0)
+		(size 17.78 5.08)
+		(margins 1.7144 1.7144 1.7144 1.7144)
+		(stroke
+			(width -0.0001)
+			(type solid)
+		)
+		(fill
+			(type none)
+		)
+		(effects
+			(font
+				(face "Times New Roman")
+				(size 2.286 2.286)
+				(thickness 0.4572)
+				(bold yes)
+				(color 0 0 0 1)
+			)
+			(justify left top)
+			(href "#10")
+		)
+	)
