File: Electronics/CM5 Nas.kicad_pcb (KiCad board)
At the start: 6 copper layers, 0 parts

Commit message: Footprints selected, Hiracicle connections created, Pcb next
Parts:
- added BT1: Battery_Cell, Battery:BatteryHolder_Keystone_3034_1x20mm, F.Cu at (-143.3, 83.5)
- added C1: 100n, Capacitor_SMD:C_0603_1608Metric, F.Cu at (-119.7, 36.9)
- added C10: 100n, Capacitor_SMD:C_0402_1005Metric, F.Cu at (-96.3, 157.4)
- added C100: 10n, Capacitor_SMD:C_0402_1005Metric, F.Cu at (-49.0, 50.8)
- added C101: 10n, Capacitor_SMD:C_0402_1005Metric, F.Cu at (-49.0, 52.7)
- added C102: 10n, Capacitor_SMD:C_0402_1005Metric, F.Cu at (-49.0, 54.7)
- added C103: 1u, Capacitor_SMD:C_0603_1608Metric, F.Cu at (-97.5, 47.1)
- added C104: 22u, Capacitor_SMD:C_1206_3216Metric, F.Cu at (-66.3, 54.2)
- added C105: 22u, Capacitor_SMD:C_1206_3216Metric, F.Cu at (-66.3, 57.6)
- added C106: 100n, Capacitor_SMD:C_0603_1608Metric, F.Cu at (-97.5, 49.6)
- added C107: 100n, Capacitor_SMD:C_0603_1608Metric, F.Cu at (-97.5, 52.1)
- added C108: 100n, Capacitor_SMD:C_0603_1608Metric, F.Cu at (-97.5, 54.6)
- added C109: 100n, Capacitor_SMD:C_0603_1608Metric, F.Cu at (-97.5, 57.1)
- added C11: 100n, Capacitor_SMD:C_0402_1005Metric, F.Cu at (-96.3, 159.4)
- added C110: 100n, Capacitor_SMD:C_0603_1608Metric, F.Cu at (-97.5, 59.6)
- added C111: 100n, Capacitor_SMD:C_0603_1608Metric, F.Cu at (-97.5, 62.2)
- added C112: 1u, Capacitor_SMD:C_0805_2012Metric, F.Cu at (-71.4, 53.4)
- added C113: 1u, Capacitor_SMD:C_0805_2012Metric, F.Cu at (-71.4, 56.4)
- added C114: 100n, Capacitor_SMD:C_0603_1608Metric, F.Cu at (-97.5, 64.7)
- added C115: 100n, Capacitor_SMD:C_0603_1608Metric, F.Cu at (-93.5, 47.1)
- added C116: 1u, Capacitor_SMD:C_0805_2012Metric, F.Cu at (-71.4, 59.4)
- added C117: 100n, Capacitor_SMD:C_0603_1608Metric, F.Cu at (-93.5, 49.6)
- added C118: 10n, Capacitor_SMD:C_0402_1005Metric, F.Cu at (-61.1, 105.0)
- added C119: 10n, Capacitor_SMD:C_0402_1005Metric, F.Cu at (-61.1, 106.9)
- added C12: 1u, Capacitor_SMD:C_1210_3225Metric, F.Cu at (-84.2, 131.8)
- added C120: 22p, Capacitor_SMD:C_0402_1005Metric, F.Cu at (-61.1, 108.9)
- added C121: 22p, Capacitor_SMD:C_0402_1005Metric, F.Cu at (-61.1, 110.9)
- added C122: 10n, Capacitor_SMD:C_0402_1005Metric, F.Cu at (-61.1, 112.8)
- added C123: 10n, Capacitor_SMD:C_0402_1005Metric, F.Cu at (-58.2, 105.0)
- added C124: 22u, Capacitor_SMD:C_1206_3216Metric, F.Cu at (-75.6, 105.6)
- added C125: 22u, Capacitor_SMD:C_1206_3216Metric, F.Cu at (-75.6, 109.0)
- added C126: 1u, Capacitor_SMD:C_0805_2012Metric, F.Cu at (-80.7, 105.5)
- added C127: 1u, Capacitor_SMD:C_0805_2012Metric, F.Cu at (-80.7, 108.5)
- added C128: 10n, Capacitor_SMD:C_0402_1005Metric, F.Cu at (-58.2, 106.9)
- added C129: 10n, Capacitor_SMD:C_0402_1005Metric, F.Cu at (-58.2, 108.9)
- added C13: 1000u, EEE0JA152UAP:EEE0JA152UAP, F.Cu at (-100.4, 149.8)
- added C130: 10n, Capacitor_SMD:C_0402_1005Metric, F.Cu at (-58.2, 110.9)
- added C131: 10n, Capacitor_SMD:C_0402_1005Metric, F.Cu at (-58.2, 112.8)
- added C132: 1u, Capacitor_SMD:C_0603_1608Metric, F.Cu at (-106.8, 105.2)
- added C133: 22u, Capacitor_SMD:C_1206_3216Metric, F.Cu at (-75.6, 112.3)
- added C134: 22u, Capacitor_SMD:C_1206_3216Metric, F.Cu at (-75.6, 115.7)
- added C135: 100n, Capacitor_SMD:C_0603_1608Metric, F.Cu at (-106.8, 107.7)
- added C136: 100n, Capacitor_SMD:C_0603_1608Metric, F.Cu at (-106.8, 110.2)
- added C137: 100n, Capacitor_SMD:C_0603_1608Metric, F.Cu at (-106.8, 112.8)
- added C138: 100n, Capacitor_SMD:C_0603_1608Metric, F.Cu at (-106.8, 115.3)
- added C139: 100n, Capacitor_SMD:C_0603_1608Metric, F.Cu at (-106.8, 117.8)
- added C14: 10u, Capacitor_SMD:C_1210_3225Metric, F.Cu at (-84.2, 136.1)
- added C140: 100n, Capacitor_SMD:C_0603_1608Metric, F.Cu at (-106.8, 120.3)
- added C141: 1u, Capacitor_SMD:C_0805_2012Metric, F.Cu at (-80.7, 111.5)
- added C142: 1u, Capacitor_SMD:C_0805_2012Metric, F.Cu at (-80.7, 114.5)
- added C143: 100n, Capacitor_SMD:C_0603_1608Metric, F.Cu at (-106.8, 122.8)
- added C144: 100n, Capacitor_SMD:C_0603_1608Metric, F.Cu at (-102.8, 105.2)
- added C145: 1u, Capacitor_SMD:C_0805_2012Metric, F.Cu at (-80.7, 117.5)
- added C146: 100n, Capacitor_SMD:C_0603_1608Metric, F.Cu at (-102.8, 107.7)
- added C147: 0u01, Capacitor_SMD:C_0402_1005Metric, F.Cu at (-27.5, 34.8)
- added C148: 100n, Capacitor_SMD:C_0603_1608Metric, F.Cu at (-23.7, 15.6)
- added C149: 22p, Capacitor_SMD:C_0402_1005Metric, F.Cu at (-27.5, 36.8)
- added C15: 10u, Capacitor_SMD:C_1210_3225Metric, F.Cu at (-84.2, 140.3)
- added C150: 22p, Capacitor_SMD:C_0402_1005Metric, F.Cu at (-27.5, 38.8)
- added C151: 100n, Capacitor_SMD:C_0603_1608Metric, F.Cu at (-23.7, 18.1)
- added C152: 100n, Capacitor_SMD:C_0603_1608Metric, F.Cu at (-23.7, 20.6)
- added C153: 0u01, Capacitor_SMD:C_0402_1005Metric, F.Cu at (-27.5, 40.7)
- added C16: 10u, Capacitor_SMD:C_1210_3225Metric, F.Cu at (-84.2, 144.6)
- added C17: 10u, Capacitor_SMD:C_1210_3225Metric, F.Cu at (-84.2, 148.8)
- added C18: 100n, Capacitor_SMD:C_0402_1005Metric, F.Cu at (-96.3, 161.3)
- added C19: 100n, Capacitor_SMD:C_0402_1005Metric, F.Cu at (-96.3, 163.3)
- added C2: 100n, Capacitor_SMD:C_0603_1608Metric, F.Cu at (-119.7, 39.4)
- added C20: 100p, Capacitor_SMD:C_0402_1005Metric, F.Cu at (-51.7, 142.7)
- added C21: 10u, Capacitor_SMD:C_0805_2012Metric, F.Cu at (-18.5, 143.2)
- added C22: 10u, EEEFK1H100UR:CAP_EEEFK1H100UR, F.Cu at (-22.4, 138.2)
- added C23: 22u, EEEFK1A220AR:CAP_EEEFK1A220AR, F.Cu at (-32.3, 144.6)
- added C24: 4n7, Capacitor_SMD:C_0402_1005Metric, F.Cu at (-51.7, 144.7)
- added C25: 3u3, Capacitor_SMD:C_0805_2012Metric, F.Cu at (-18.5, 146.2)
- added C26: 4n7, Capacitor_SMD:C_0402_1005Metric, F.Cu at (-51.7, 146.6)
- added C27: 4n7, Capacitor_SMD:C_0402_1005Metric, F.Cu at (-51.7, 148.6)
- added C28: 22u, EEEFK1A220AR:CAP_EEEFK1A220AR, F.Cu at (-32.3, 150.5)
- added C29: 47n, Capacitor_SMD:C_0402_1005Metric, F.Cu at (-51.7, 150.6)
- added C3: 10u, Capacitor_SMD:C_0805_2012Metric, F.Cu at (-153.4, 127.3)
- added C30: 22u, EEEFK1A220AR:CAP_EEEFK1A220AR, F.Cu at (-32.3, 156.3)
- added C31: 47n, Capacitor_SMD:C_0402_1005Metric, F.Cu at (-51.7, 152.6)
- added C32: 47n, Capacitor_SMD:C_0402_1005Metric, F.Cu at (-48.9, 142.7)
- added C33: 22u, EEEFK1A220AR:CAP_EEEFK1A220AR, F.Cu at (-32.3, 162.2)
- added C34: 4n7, Capacitor_SMD:C_0402_1005Metric, F.Cu at (-48.9, 144.7)
- added C35: 4n7, Capacitor_SMD:C_0402_1005Metric, F.Cu at (-48.9, 146.6)
- added C36: 4n7, Capacitor_SMD:C_0402_1005Metric, F.Cu at (-48.9, 148.6)
- added C37: 4n7, Capacitor_SMD:C_0402_1005Metric, F.Cu at (-48.9, 150.6)
- added C38: 100n, Capacitor_SMD:C_0603_1608Metric, F.Cu at (-51.1, 127.9)
- added C39: 100u, EEE_FTH101XAP:CAP_EEEFTH101XAP, F.Cu at (-22.4, 130.7)
- added C4: 1u, Capacitor_SMD:C_1210_3225Metric, F.Cu at (-89.8, 131.8)
- added C40: 100n, Capacitor_SMD:C_0402_1005Metric, F.Cu at (-48.9, 152.6)
- added C41: 4u7, Capacitor_SMD:C_0805_2012Metric, F.Cu at (-18.5, 149.2)
- added C42: 4n7, Capacitor_SMD:C_0402_1005Metric, F.Cu at (-46.0, 142.7)
- added C43: 4n7, Capacitor_SMD:C_0402_1005Metric, F.Cu at (-46.0, 144.7)
- added C44: 4u7, Capacitor_SMD:C_0805_2012Metric, F.Cu at (-18.5, 152.2)
- added C45: 4u7, Capacitor_SMD:C_0805_2012Metric, F.Cu at (-18.5, 155.3)
- added C46: 100p, Capacitor_SMD:C_0402_1005Metric, F.Cu at (-46.0, 146.6)
- added C47: 100p, Capacitor_SMD:C_0402_1005Metric, F.Cu at (-46.0, 148.6)
- added C48: 2u2, Capacitor_SMD:C_0603_1608Metric, F.Cu at (-51.1, 130.4)
- added C49: 4u7, Capacitor_SMD:C_0805_2012Metric, F.Cu at (-18.5, 158.3)
- added C5: 1000u, EEE0JA152UAP:EEE0JA152UAP, F.Cu at (-100.4, 136.4)
- added C50: 100n, Capacitor_SMD:C_0603_1608Metric, F.Cu at (-51.1, 132.9)
- added C51: 1n, Capacitor_SMD:C_0402_1005Metric, F.Cu at (-46.0, 150.6)
- added C52: 100n, Capacitor_SMD:C_0402_1005Metric, F.Cu at (-22.3, 107.3)
- added C53: 100n, Capacitor_SMD:C_0402_1005Metric, F.Cu at (-22.3, 109.2)
- added C54: 100n, Capacitor_SMD:C_0603_1608Metric, F.Cu at (-26.1, 73.7)
- added C55: 100n, Capacitor_SMD:C_0603_1608Metric, F.Cu at (-26.1, 76.2)
- added C56: 100n, Capacitor_SMD:C_0603_1608Metric, F.Cu at (-26.1, 78.7)
- added C57: 100n, Capacitor_SMD:C_0603_1608Metric, F.Cu at (-26.1, 81.2)
- added C58: 100n, Capacitor_SMD:C_0603_1608Metric, F.Cu at (-26.1, 83.8)
- added C59: 100n, Capacitor_SMD:C_0603_1608Metric, F.Cu at (-26.1, 86.3)
- added C6: 10u, Capacitor_SMD:C_1210_3225Metric, F.Cu at (-89.8, 136.1)
- added C60: 100n, Capacitor_SMD:C_0402_1005Metric, F.Cu at (-22.3, 111.2)
- added C61: 100n, Capacitor_SMD:C_0402_1005Metric, F.Cu at (-22.3, 113.2)
- added C62: 100n, Capacitor_SMD:C_0402_1005Metric, F.Cu at (-19.4, 107.3)
- added C63: 100n, Capacitor_SMD:C_0402_1005Metric, F.Cu at (-19.4, 109.2)
- added C64: 100n, Capacitor_SMD:C_0402_1005Metric, F.Cu at (-19.4, 111.2)
- added C65: 100n, Capacitor_SMD:C_0603_1608Metric, F.Cu at (-26.1, 88.8)
- added C66: 100n, Capacitor_SMD:C_0603_1608Metric, F.Cu at (-26.1, 91.3)
- added C67: 100n, Capacitor_SMD:C_0603_1608Metric, F.Cu at (-26.1, 93.8)
- added C68: 100n, Capacitor_SMD:C_0603_1608Metric, F.Cu at (-22.1, 73.7)
- added C69: 100n, Capacitor_SMD:C_0603_1608Metric, F.Cu at (-22.1, 76.2)
- added C7: 10u, Capacitor_SMD:C_1210_3225Metric, F.Cu at (-89.8, 140.3)
- added C70: 100n, Capacitor_SMD:C_0603_1608Metric, F.Cu at (-22.1, 78.7)
- added C71: 100n, Capacitor_SMD:C_0402_1005Metric, F.Cu at (-19.4, 113.2)
- added C72: 100n, Capacitor_SMD:C_0402_1005Metric, F.Cu at (-16.5, 107.3)
- added C73: 10u, Capacitor_SMD:C_0805_2012Metric, F.Cu at (-25.9, 107.8)
- added C74: 0u47, Capacitor_SMD:C_0603_1608Metric, F.Cu at (-22.1, 81.2)
- added C75: 100n, Capacitor_SMD:C_0402_1005Metric, F.Cu at (-16.5, 109.2)
- added C76: 0u47, Capacitor_SMD:C_0603_1608Metric, F.Cu at (-22.1, 83.8)
- added C77: 10u, Capacitor_SMD:C_0805_2012Metric, F.Cu at (-25.9, 110.8)
- added C78: 100n, Capacitor_SMD:C_0603_1608Metric, F.Cu at (-22.1, 86.3)
- added C79: 100n, Capacitor_SMD:C_0603_1608Metric, F.Cu at (-22.1, 88.8)
- added C8: 10u, Capacitor_SMD:C_1210_3225Metric, F.Cu at (-89.8, 144.6)
- added C80: 100n, Capacitor_SMD:C_0603_1608Metric, F.Cu at (-22.1, 91.3)
- added C81: 100n, Capacitor_SMD:C_0603_1608Metric, F.Cu at (-22.1, 93.8)
- added C82: 100n, Capacitor_SMD:C_0603_1608Metric, F.Cu at (-18.1, 73.7)
- added C83: 100n, Capacitor_SMD:C_0603_1608Metric, F.Cu at (-18.1, 76.2)
- added C84: 100n, Capacitor_SMD:C_0402_1005Metric, F.Cu at (-16.5, 111.2)
- added C85: 100n, Capacitor_SMD:C_0402_1005Metric, F.Cu at (-16.5, 113.2)
- added C86: 47u, Capacitor_SMD:C_0805_2012Metric, F.Cu at (-25.9, 113.8)
- added C87: 47u, Capacitor_SMD:C_0805_2012Metric, F.Cu at (-25.9, 116.8)
- added C88: 47u, Capacitor_SMD:C_0805_2012Metric, F.Cu at (-25.9, 119.8)
- added C89: 22p, Capacitor_SMD:C_0402_1005Metric, F.Cu at (-51.8, 46.8)
- added C9: 10u, Capacitor_SMD:C_1210_3225Metric, F.Cu at (-89.8, 148.8)
- added C90: 22p, Capacitor_SMD:C_0402_1005Metric, F.Cu at (-51.8, 48.8)
- added C91: 10n, Capacitor_SMD:C_0402_1005Metric, F.Cu at (-51.8, 50.8)
- added C92: 10n, Capacitor_SMD:C_0402_1005Metric, F.Cu at (-51.8, 52.7)
- added C93: 10n, Capacitor_SMD:C_0402_1005Metric, F.Cu at (-51.8, 54.7)
- added C94: 10n, Capacitor_SMD:C_0402_1005Metric, F.Cu at (-49.0, 46.8)
- added C95: 22u, Capacitor_SMD:C_1206_3216Metric, F.Cu at (-66.3, 47.5)
- added C96: 1u, Capacitor_SMD:C_0805_2012Metric, F.Cu at (-71.4, 47.4)
- added C97: 22u, Capacitor_SMD:C_1206_3216Metric, F.Cu at (-66.3, 50.9)
- added C98: 1u, Capacitor_SMD:C_0805_2012Metric, F.Cu at (-71.4, 50.4)
- added C99: 10n, Capacitor_SMD:C_0402_1005Metric, F.Cu at (-49.0, 48.8)
- added D1: LED Green, LED_SMD:LED_0603_1608Metric, F.Cu at (-112.8, 103.3)
- added D10: LED Green, LED_SMD:LED_0603_1608Metric, F.Cu at (-13.5, 115.5)
- added D11: LED Green, LED_SMD:LED_0603_1608Metric, F.Cu at (-13.5, 118.1)
- added D12: LED Green, LED_SMD:LED_0603_1608Metric, F.Cu at (-13.5, 120.7)
- added D13: LED Green, LED_SMD:LED_0603_1608Metric, F.Cu at (-13.5, 123.2)
- added D14: LED Green, LED_SMD:LED_0603_1608Metric, F.Cu at (-67.1, 60.5)
- added D15: LED Green, LED_SMD:LED_0603_1608Metric, F.Cu at (-67.1, 63.1)
- added D16: LED Green, LED_SMD:LED_0603_1608Metric, F.Cu at (-67.1, 65.7)
- added D17: LED Green, LED_SMD:LED_0603_1608Metric, F.Cu at (-67.1, 68.3)
- added D18: LED Green, LED_SMD:LED_0603_1608Metric, F.Cu at (-76.4, 118.7)
- added D19: LED Green, LED_SMD:LED_0603_1608Metric, F.Cu at (-76.4, 121.2)
- added D2: LED Red, LED_SMD:LED_0603_1608Metric, F.Cu at (-112.8, 105.9)
- added D20: LED Green, LED_SMD:LED_0603_1608Metric, F.Cu at (-76.4, 123.8)
- added D21: LED Green, LED_SMD:LED_0603_1608Metric, F.Cu at (-76.4, 126.4)
- added D3: LED Green, LED_SMD:LED_0603_1608Metric, F.Cu at (-95.7, 165.6)
- added D4: D_TVS, SMBJ12A:SMBJ12A, F.Cu at (-104.8, 159.2)
- added D5: D_TVS, SMBJ5.0A:SMBJ5.0A, F.Cu at (-104.8, 164.9)
- added D6: LED Green, LED_SMD:LED_0603_1608Metric, F.Cu at (-95.7, 168.2)
- added D7: LED Green, LED_SMD:LED_0603_1608Metric, F.Cu at (-42.5, 158.7)
- added D8: LED Green, LED_SMD:LED_0603_1608Metric, F.Cu at (-42.5, 161.2)
- added D9: LED Green, LED_SMD:LED_0603_1608Metric, F.Cu at (-42.5, 163.8)
- added F1: Polyfuse, RGEF1200:RGEF1200, F.Cu at (-76.7, 132.2)
- added F2: Polyfuse, RGEF1200:RGEF1200, F.Cu at (-76.7, 138.5)
- added H1: MountingHole, MountingHole:MountingHole_2.7mm_M2.5, F.Cu at (-40.8, 47.2)
- added H2: MountingHole, MountingHole:MountingHole_2.7mm_M2.5, F.Cu at (-40.8, 53.5)
- added H3: MountingHole, MountingHole:MountingHole_2.7mm_M2.5, F.Cu at (-34.5, 47.2)
- added H4: MountingHole, MountingHole:MountingHole_2.7mm_M2.5, F.Cu at (-34.5, 53.5)
- added H5: MountingHole, MountingHole:MountingHole_2.7mm_M2.5, F.Cu at (-28.3, 47.2)
- added H6: MountingHole, MountingHole:MountingHole_2.7mm_M2.5, F.Cu at (-28.3, 53.5)
- added H7: MountingHole, MountingHole:MountingHole_2.7mm_M2.5, F.Cu at (-22.0, 47.2)
- added H8: MountingHole, MountingHole:MountingHole_2.7mm_M2.5, F.Cu at (-22.0, 53.5)
- added IC1: TPS65251-1RHAR, TPS65251-1RHAR:QFN50P600X600X100-41N-D, F.Cu at (-49.0, 157.7)
- added IC2: MAX20008AFOC_VY+T, MAX20008AFOC_VY+T:MAX20008AFOCVYT, F.Cu at (-40.9, 153.6)
- added IC3: LM61480Q3RPHRQ1, LIB_LM61480Q3RPHRQ1:LM62460QRPHRQ1, F.Cu at (-13.4, 99.0)
- added IC4: USB2512B-AEZG, USB2512B-AEZG:QFN50P600X600X100-37N-D, F.Cu at (-39.8, 38.0)
- added J1: THD-02-R, Connector_PinHeader_2.54mm:PinHeader_2x02_P2.54mm_Vertical, F.Cu at (-115.4, 38.0)
- added J10: JST_SHBM04B-SRSS-TB, Connector_JST:JST_SH_BM04B-SRSS-TB_1x04-1MP_P1.00mm_Vertical, F.Cu at (-131.1, 97.6)
- added J11: JST_SHBM04B-SRSS-TB, Connector_JST:JST_SH_BM04B-SRSS-TB_1x04-1MP_P1.00mm_Vertical, F.Cu at (-131.1, 103.9)
- added J12: JST_SHBM04B-SRSS-TB, Connector_JST:JST_SH_BM04B-SRSS-TB_1x04-1MP_P1.00mm_Vertical, F.Cu at (-131.1, 110.1)
- added J13: JST_SHBM04B-SRSS-TB, Connector_JST:JST_SH_BM04B-SRSS-TB_1x04-1MP_P1.00mm_Vertical, F.Cu at (-131.1, 116.4)
- added J14: JST_SHBM04B-SRSS-TB, Connector_JST:JST_SH_BM04B-SRSS-TB_1x04-1MP_P1.00mm_Vertical, F.Cu at (-131.1, 122.6)
- added J15: 4DB-P108-03, 4DB-P108-03:4DBP10803, F.Cu at (-86.0, 154.8)
- added J16: Bus_M.2_Socket_M, 2199119-5:21991195, F.Cu at (-40.7, 79.4)
- added J17: Bus_M.2_Socket_M, 2199119-5:21991195, F.Cu at (-40.7, 92.5)
- added J18: Bus_M.2_Socket_M, 2199119-5:21991195, F.Cu at (-40.7, 105.5)
- added J19: Bus_M.2_Socket_M, 2199119-5:21991195, F.Cu at (-40.7, 118.6)
- added J2: HDMI_A, 10029449-111RLF:AMPHENOL_10029449-111RLF, F.Cu at (-112.0, 22.4)
- added J20: 47018-2000, 47018-2000:MOLEX_47018-2000, F.Cu at (-78.5, 20.0)
- added J21: 47018-2000, 47018-2000:MOLEX_47018-2000, F.Cu at (-78.5, 35.8)
- added J22: 47018-2000, 47018-2000:MOLEX_47018-2000, F.Cu at (-87.8, 78.2)
- added J23: 47018-2000, 47018-2000:MOLEX_47018-2000, F.Cu at (-87.8, 93.9)
- added J24: USB_A_Stacked, Connector_USB:USB_A_Wuerth_61400826021_Horizontal_Stacked, F.Cu at (-38.3, 17.2)
- added J3: Conn_01x22_Female, Connector_FFC-FPC:Hirose_FH12-22S-0.5SH_1x22-1MP_P0.50mm_Horizontal, F.Cu at (-112.6, 30.2)
- added J4: THD-20-R, Connector_PinHeader_2.54mm:PinHeader_2x20_P2.54mm_Vertical, F.Cu at (-160.5, 74.8)
- added J5: RJ45_RB1-125B8G1A, Connector_RJ:RJ45_UDE_RB1-125B8G1A, F.Cu at (-151.3, 97.5)
- added J6: Conn_01x07, Connector_JST:JST_GH_SM07B-GHS-TB_1x07-1MP_P1.25mm_Horizontal, F.Cu at (-148.5, 122.0)
- added J7: Micro_SD_Card_Det, DM3AT-SF-PEJM5:DM3ATSFPEJM5, F.Cu at (-122.0, 82.6)
- added J8: Conn_01x04, PRT-14417:SPARKFUN_PRT-14417, F.Cu at (-115.4, 98.9)
- added J9: Conn_02x07_Odd_Even, Connector_PinHeader_2.54mm:PinHeader_2x07_P2.54mm_Vertical, F.Cu at (-124.4, 96.8)
- added JP1: 3P_JUMPER, Connector_PinHeader_2.54mm:PinHeader_1x03_P2.54mm_Vertical, F.Cu at (-61.2, 58.4)
- added JP2: 3P_JUMPER, Connector_PinHeader_2.54mm:PinHeader_1x03_P2.54mm_Vertical, F.Cu at (-56.6, 58.4)
- added JP3: 3P_JUMPER, Connector_PinHeader_2.54mm:PinHeader_1x03_P2.54mm_Vertical, F.Cu at (-70.5, 116.5)
- added JP4: 3P_JUMPER, Connector_PinHeader_2.54mm:PinHeader_1x03_P2.54mm_Vertical, F.Cu at (-65.9, 116.5)
- added L1: 4u7, SRN5040-4R7M:INDPM5050X400N, F.Cu at (-24.6, 145.1)
- added L2: 4u7, SRN5040-4R7M:INDPM5050X400N, F.Cu at (-24.6, 151.8)
- added L3: 4u7, SRN5040-4R7M:INDPM5050X400N, F.Cu at (-24.6, 158.6)
- added L4: 1u, SRN5040TA-1R0M:SRN5040TA1R0M, F.Cu at (-40.4, 145.8)
- added L5: 2u2, SRN5040-2R2Y:SRN50402R2Y, F.Cu at (-19.6, 118.2)
- added Module1: ComputeModule5-CM5, cm5:Raspberry-Pi-5-Compute-Module, F.Cu at (-158.7, 66.4)
- added Q1: PMOS, BSS84AKW115:BSS84AKW115, F.Cu at (-117.0, 110.7)
- added Q10: NPN, MMBT3904:P200_SOT-23, F.Cu at (-86.4, 105.2)
- added Q11: PMOS, AOSS21311C:SOT95P237X117-3N, F.Cu at (-90.2, 106.3)
- added Q12: NPN, MMBT3904:P200_SOT-23, F.Cu at (-86.4, 109.6)
- added Q13: PMOS, AOSS21311C:SOT95P237X117-3N, F.Cu at (-90.2, 110.8)
- added Q14: PMOS, AOSS21311C:SOT95P237X117-3N, F.Cu at (-90.2, 115.4)
- added Q15: NPN, MMBT3904:P200_SOT-23, F.Cu at (-86.4, 114.1)
- added Q16: NPN, MMBT3904:P200_SOT-23, F.Cu at (-86.4, 118.5)
- added Q17: PMOS, AOSS21311C:SOT95P237X117-3N, F.Cu at (-90.2, 120.0)
- added Q2: NPN, MMBT3904:P200_SOT-23, F.Cu at (-77.2, 47.0)
- added Q3: PMOS, AOSS21311C:SOT95P237X117-3N, F.Cu at (-81.0, 48.1)
- added Q4: NPN, MMBT3904:P200_SOT-23, F.Cu at (-77.2, 51.5)
- added Q5: PMOS, AOSS21311C:SOT95P237X117-3N, F.Cu at (-81.0, 52.7)
- added Q6: PMOS, AOSS21311C:SOT95P237X117-3N, F.Cu at (-81.0, 57.3)
- added Q7: NPN, MMBT3904:P200_SOT-23, F.Cu at (-77.2, 55.9)
- added Q8: NPN, MMBT3904:P200_SOT-23, F.Cu at (-77.2, 60.4)
- added Q9: PMOS, AOSS21311C:SOT95P237X117-3N, F.Cu at (-81.0, 61.9)
- added R1: 2K2 1%, Resistor_SMD:R_0603_1608Metric, F.Cu at (-119.7, 42.0)
- added R10: nf, Resistor_SMD:R_0805_2012Metric_Pad1.20x1.40mm_HandSolder, F.Cu at (-117.2, 106.5)
- added R11: 2K2, Resistor_SMD:R_0603_1608Metric, F.Cu at (-79.4, 143.6)
- added R12: 620, Resistor_SMD:R_0603_1608Metric, F.Cu at (-79.4, 146.1)
- added R13: 20k, Resistor_SMD:R_0603_1608Metric, F.Cu at (-51.1, 135.4)
- added R14: 80K6, Resistor_SMD:R_0603_1608Metric, F.Cu at (-51.1, 137.9)
- added R15: 150k, Resistor_SMD:R_0603_1608Metric, F.Cu at (-51.1, 140.5)
- added R16: 40K2, Resistor_SMD:R_0603_1608Metric, F.Cu at (-47.1, 127.9)
- added R17: 270, Resistor_SMD:R_0603_1608Metric, F.Cu at (-47.1, 130.4)
- added R18: 270, Resistor_SMD:R_0603_1608Metric, F.Cu at (-47.1, 132.9)
- added R19: 1K, Resistor_SMD:R_0603_1608Metric, F.Cu at (-47.1, 135.4)
- added R2: 2K2 1%, Resistor_SMD:R_0603_1608Metric, F.Cu at (-119.7, 44.5)
- added R20: 40K2, Resistor_SMD:R_0603_1608Metric, F.Cu at (-47.1, 137.9)
- added R21: 40K2, Resistor_SMD:R_0603_1608Metric, F.Cu at (-47.1, 140.5)
- added R22: 120k, Resistor_SMD:R_0603_1608Metric, F.Cu at (-43.1, 127.9)
- added R23: 150k, Resistor_SMD:R_0603_1608Metric, F.Cu at (-43.1, 130.4)
- added R24: 20K, Resistor_SMD:R_0603_1608Metric, F.Cu at (-43.1, 132.9)
- added R25: 12K7, Resistor_SMD:R_0603_1608Metric, F.Cu at (-43.1, 135.4)
- added R26: 80K6, Resistor_SMD:R_0603_1608Metric, F.Cu at (-43.1, 137.9)
- added R27: 383k, Resistor_SMD:R_0603_1608Metric, F.Cu at (-43.1, 140.5)
- added R28: 20k, Resistor_SMD:R_0603_1608Metric, F.Cu at (-39.1, 127.9)
- added R29: 20k, Resistor_SMD:R_0603_1608Metric, F.Cu at (-39.1, 130.4)
- added R3: 1K, Resistor_SMD:R_0603_1608Metric, F.Cu at (-114.1, 115.6)
- added R30: 22K, Resistor_SMD:R_0603_1608Metric, F.Cu at (-39.1, 132.9)
- added R31: 12k, Resistor_SMD:R_0603_1608Metric, F.Cu at (-39.1, 135.4)
- added R32: 10K, Resistor_SMD:R_0603_1608Metric, F.Cu at (-18.1, 78.7)
- added R33: 10K, Resistor_SMD:R_0603_1608Metric, F.Cu at (-18.1, 81.2)
- added R34: 10K, Resistor_SMD:R_0603_1608Metric, F.Cu at (-18.1, 83.8)
- added R35: 10K, Resistor_SMD:R_0603_1608Metric, F.Cu at (-18.1, 86.3)
- added R36: 10K, Resistor_SMD:R_0603_1608Metric, F.Cu at (-18.1, 88.8)
- added R37: 10k, Resistor_SMD:R_0603_1608Metric, F.Cu at (-18.1, 91.3)
- added R38: 1K, Resistor_SMD:R_0603_1608Metric, F.Cu at (-18.1, 93.8)
- added R39: 1K, Resistor_SMD:R_0603_1608Metric, F.Cu at (-14.1, 73.7)
- added R4: 1K, Resistor_SMD:R_0603_1608Metric, F.Cu at (-114.1, 118.1)
- added R40: 1K, Resistor_SMD:R_0603_1608Metric, F.Cu at (-14.1, 76.2)
- added R41: 1K, Resistor_SMD:R_0603_1608Metric, F.Cu at (-14.1, 78.7)
- added R42: 12K1, Resistor_SMD:R_0603_1608Metric, F.Cu at (-14.1, 81.2)
- added R43: 12K1, Resistor_SMD:R_0603_1608Metric, F.Cu at (-14.1, 83.8)
- added R44: 1k, Resistor_SMD:R_0603_1608Metric, F.Cu at (-14.1, 86.3)
- added R45: 1k, Resistor_SMD:R_0603_1608Metric, F.Cu at (-14.1, 88.8)
- added R46: 1k, Resistor_SMD:R_0603_1608Metric, F.Cu at (-14.1, 91.3)
- added R47: 1k, Resistor_SMD:R_0603_1608Metric, F.Cu at (-14.1, 93.8)
- added R48: 12K, Resistor_SMD:R_0603_1608Metric, F.Cu at (-93.5, 52.1)
- added R49: 100K, Resistor_SMD:R_0603_1608Metric, F.Cu at (-93.5, 54.6)
- added R5: 1K, Resistor_SMD:R_0603_1608Metric, F.Cu at (-114.1, 120.6)
- added R50: 100K, Resistor_SMD:R_0603_1608Metric, F.Cu at (-93.5, 57.1)
- added R51: 100K, Resistor_SMD:R_0603_1608Metric, F.Cu at (-93.5, 59.6)
- added R52: 100K, Resistor_SMD:R_0603_1608Metric, F.Cu at (-93.5, 62.2)
- added R53: 12K, Resistor_SMD:R_0603_1608Metric, F.Cu at (-93.5, 64.7)
- added R54: 4K7, Resistor_SMD:R_0603_1608Metric, F.Cu at (-89.5, 47.1)
- added R55: 100K, Resistor_SMD:R_0603_1608Metric, F.Cu at (-89.5, 49.6)
- added R56: 100K, Resistor_SMD:R_0603_1608Metric, F.Cu at (-89.5, 52.1)
- added R57: 100K, Resistor_SMD:R_0603_1608Metric, F.Cu at (-89.5, 54.6)
- added R58: 100K, Resistor_SMD:R_0603_1608Metric, F.Cu at (-89.5, 57.1)
- added R59: 10, Resistor_SMD:R_0603_1608Metric, F.Cu at (-89.5, 59.6)
- added R6: 1k, Resistor_SMD:R_0603_1608Metric, F.Cu at (-114.1, 123.1)
- added R60: 4K7, Resistor_SMD:R_0603_1608Metric, F.Cu at (-89.5, 62.2)
- added R61: 4K7 1%, Resistor_SMD:R_0603_1608Metric, F.Cu at (-89.5, 64.7)
- added R62: 270, Resistor_SMD:R_0603_1608Metric, F.Cu at (-85.5, 47.1)
- added R63: 270, Resistor_SMD:R_0603_1608Metric, F.Cu at (-85.5, 49.6)
- added R64: 270, Resistor_SMD:R_0603_1608Metric, F.Cu at (-85.5, 52.1)
- added R65: 270, Resistor_SMD:R_0603_1608Metric, F.Cu at (-85.5, 54.6)
- added R66: 12K, Resistor_SMD:R_0603_1608Metric, F.Cu at (-102.8, 110.2)
- added R67: 100K, Resistor_SMD:R_0603_1608Metric, F.Cu at (-102.8, 112.8)
- added R68: 100K, Resistor_SMD:R_0603_1608Metric, F.Cu at (-102.8, 115.3)
- added R69: 100K, Resistor_SMD:R_0603_1608Metric, F.Cu at (-102.8, 117.8)
- added R7: 4K7, Resistor_SMD:R_0603_1608Metric, F.Cu at (-114.1, 125.6)
- added R70: 100K, Resistor_SMD:R_0603_1608Metric, F.Cu at (-102.8, 120.3)
- added R71: 4K7, Resistor_SMD:R_0603_1608Metric, F.Cu at (-102.8, 122.8)
- added R72: 12K, Resistor_SMD:R_0603_1608Metric, F.Cu at (-98.7, 105.2)
- added R73: 100K, Resistor_SMD:R_0603_1608Metric, F.Cu at (-98.7, 107.7)
- added R74: 100K, Resistor_SMD:R_0603_1608Metric, F.Cu at (-98.7, 110.2)
- added R75: 100K, Resistor_SMD:R_0603_1608Metric, F.Cu at (-98.7, 112.8)
- added R76: 100K, Resistor_SMD:R_0603_1608Metric, F.Cu at (-98.7, 115.3)
- added R77: 10, Resistor_SMD:R_0603_1608Metric, F.Cu at (-98.7, 117.8)
- added R78: 4K7, Resistor_SMD:R_0603_1608Metric, F.Cu at (-98.7, 120.3)
- added R79: 4K7 1%, Resistor_SMD:R_0603_1608Metric, F.Cu at (-98.7, 122.8)
- added R8: 4K7, Resistor_SMD:R_0603_1608Metric, F.Cu at (-114.1, 128.2)
- added R80: 270, Resistor_SMD:R_0603_1608Metric, F.Cu at (-94.7, 105.2)
- added R81: 270, Resistor_SMD:R_0603_1608Metric, F.Cu at (-94.7, 107.7)
- added R82: 270, Resistor_SMD:R_0603_1608Metric, F.Cu at (-94.7, 110.2)
- added R83: 270, Resistor_SMD:R_0603_1608Metric, F.Cu at (-94.7, 112.8)
- added R84: 1K, Resistor_SMD:R_0603_1608Metric, F.Cu at (-23.7, 23.1)
- added R85: 330, Resistor_SMD:R_0603_1608Metric, F.Cu at (-23.7, 25.6)
- added R86: 12K, Resistor_SMD:R_0603_1608Metric, F.Cu at (-23.7, 28.1)
- added R9: 0R, Resistor_SMD:R_0805_2012Metric_Pad1.20x1.40mm_HandSolder, F.Cu at (-117.2, 103.5)
- added SW1: Right angle Tact button, Button_Switch_THT:SW_Tactile_SPST_Angled_PTS645Vx58-2LFS, F.Cu at (-123.7, 120.7)
- added TP1: TestPoint, TestPoint:TestPoint_Pad_1.0x1.0mm, F.Cu at (-112.9, 109.5)
- added TP10: TestPoint, TestPoint:TestPoint_Pad_1.0x1.0mm, F.Cu at (-29.5, 136.5)
- added TP11: TestPoint, TestPoint:TestPoint_Pad_1.0x1.0mm, F.Cu at (-29.5, 139.6)
- added TP12: TestPoint, TestPoint:TestPoint_Pad_1.0x1.0mm, F.Cu at (-13.6, 112.4)
- added TP2: TestPoint, TestPoint:TestPoint_Pad_1.0x1.0mm, F.Cu at (-112.9, 112.5)
- added TP3: TestPoint, TestPoint:TestPoint_Pad_1.0x1.0mm, F.Cu at (-99.3, 157.9)
- added TP4: TestPoint, TestPoint:TestPoint_Pad_1.0x1.0mm, F.Cu at (-99.3, 161.0)
- added TP5: TestPoint, TestPoint:TestPoint_Pad_1.0x1.0mm, F.Cu at (-99.3, 164.1)
- added TP6: TestPoint, TestPoint:TestPoint_Pad_1.0x1.0mm, F.Cu at (-35.6, 136.5)
- added TP7: TestPoint, TestPoint:TestPoint_Pad_1.0x1.0mm, F.Cu at (-35.6, 139.6)
- added TP8: TestPoint, TestPoint:TestPoint_Pad_1.0x1.0mm, F.Cu at (-32.5, 136.5)
- added TP9: TestPoint, TestPoint:TestPoint_Pad_1.0x1.0mm, F.Cu at (-32.5, 139.6)
- added U1: RT9742SNGV, Package_TO_SOT_SMD:TSOT-23_HandSoldering, F.Cu at (-107.0, 38.1)
- added U10: JMS561, Package_DFN_QFN:QFN-64-1EP_8x8mm_P0.4mm_EP6.5x6.5mm, F.Cu at (-58.4, 51.0)
- added U11: W25X40CLSN, Package_SO:SOIC-8_3.9x4.9mm_P1.27mm, F.Cu at (-59.4, 117.6)
- added U12: JMS561, Package_DFN_QFN:QFN-64-1EP_8x8mm_P0.4mm_EP6.5x6.5mm, F.Cu at (-67.7, 109.1)
- added U2: TPD4EUSB30, Package_SON:USON-10_2.5x1.0mm_P0.5mm, F.Cu at (-139.9, 120.6)
- added U3: TPD4EUSB30, Package_SON:USON-10_2.5x1.0mm_P0.5mm, F.Cu at (-137.1, 120.6)
- added U4: 74LVC1G07SE-7, Package_TO_SOT_SMD:SOT-353_SC-70-5, F.Cu at (-160.7, 127.3)
- added U5: RT9742GGJ5, Package_TO_SOT_SMD:SOT-23-5, F.Cu at (-138.8, 125.0)
- added U6: AMS1117-3.3, Package_TO_SOT_SMD:SOT-223-3_TabPin2, F.Cu at (-32.2, 130.9)
- added U7: ASEK-32.768KHZ-L-R-T, Crystal:Crystal_SMD_3225-4Pin_3.2x2.5mm, F.Cu at (-12.5, 108.6)
- added U8: ASM1184, Package_DFN_QFN:QFN-64-1EP_9x9mm_P0.5mm_EP5.2x5.2mm, F.Cu at (-22.5, 100.7)
- added U9: W25X40CLSN, Package_SO:SOIC-8_3.9x4.9mm_P1.27mm, F.Cu at (-50.1, 59.5)
- added Y1: 30MHz, ABM8-30.000MHZ-B2-T:ABM810000MHZ12D2W, F.Cu at (-51.0, 65.7)
- added Y2: 30MHz, ABM8-30.000MHZ-B2-T:ABM810000MHZ12D2W, F.Cu at (-60.3, 123.8)
- added Y3: 30MHz, ABM8-30.000MHZ-B2-T:ABM810000MHZ12D2W, F.Cu at (-32.3, 36.8)
