File: Electronics/CM5 Nas.kicad_pcb (KiCad board)
At the start: 4 copper layers, 352 parts, among them IC1 TPS65251-1RHAR, IC2 MAX20008AFOC_VY+T, IC3 LM61480Q3RPHRQ1, IC4 USB2512B-AEZG, J1 THD-02-R, J10 JST_SHBM04B-SRSS-TB, J11 JST_SHBM04B-SRSS-TB, J12 JST_SHBM04B-SRSS-TB, J13 JST_SHBM04B-SRSS-TB, J14 JST_SHBM04B-SRSS-TB, J15 4DB-P108-03, J2 HDMI_A, J20 47018-2000, J21 47018-2000, J22 47018-2000, J23 47018-2000, J24 USB_A_Stacked, J3 Conn_01x22_Female, J4 THD-20-R, J5 RJ45_RB1-125B8G1A, J6 Conn_01x07, J7 Micro_SD_Card_Det, J8 Conn_01x04, J9 Conn_02x07_Odd_Even, Q1 PMOS, Q10 NPN, Q11 PMOS, Q12 NPN, Q13 PMOS, Q14 PMOS, Q15 NPN, Q16 NPN, Q17 PMOS, Q2 NPN, Q3 PMOS, Q4 NPN, Q5 PMOS, Q6 PMOS, Q7 NPN, Q8 NPN, Q9 PMOS, SW1 Right angle Tact button, U1 RT9742SNGV, U10 JMS561, U11 W25X40CLSN, U12 JMS561, U2 TPD4EUSB30, U3 TPD4EUSB30, U4 74LVC1G07SE-7, U5 RT9742GGJ5, U6 AMS1117-3.3, U7 ASEK-32.768KHZ-L-R-T, U8 ASM1184, U9 W25X40CLSN, Y1 30MHz, Y2 30MHz, Y3 30MHz

Commit message: Changed sata port
Parts:
- removed H6, H7, H8: MountingHole, MountingHole:MountingHole_2.7mm_M2.5
- removed the J1 at (-115.4, 38.0)
- removed the J22 at (-87.8, 78.2)
- removed J23: 47018-2000, 47018-2000:MOLEX_47018-2000
- removed the J4 at (-160.5, 74.8)
- removed the R1 at (-119.7, 42.0)
- removed the R2 at (-119.7, 44.5)
- removed SW1: Right angle Tact button, Button_Switch_THT:SW_Tactile_SPST_Angled_PTS645Vx58-2LFS
- added C125: 22u, Capacitor_SMD:C_1206_3216Metric, F.Cu at (-102.7, 163.8)
- added C126: 22u, Capacitor_SMD:C_1206_3216Metric, F.Cu at (-102.7, 167.2)
- added C128: 10n, Capacitor_SMD:C_0402_1005Metric, F.Cu at (-106.9, 163.1)
- added C129: 10n, Capacitor_SMD:C_0402_1005Metric, F.Cu at (-106.9, 165.1)
- added C130: 10n, Capacitor_SMD:C_0402_1005Metric, F.Cu at (-106.9, 167.1)
- added C131: 10n, Capacitor_SMD:C_0402_1005Metric, F.Cu at (-106.9, 169.1)
- added C133: 22u, Capacitor_SMD:C_1206_3216Metric, F.Cu at (-102.7, 170.5)
- added C135: 22u, Capacitor_SMD:C_1206_3216Metric, F.Cu at (-102.7, 173.9)
- added C140: 10n, Capacitor_SMD:C_0402_1005Metric, F.Cu at (-106.9, 171.0)
- added C141: 10n, Capacitor_SMD:C_0402_1005Metric, F.Cu at (-106.9, 173.0)
- added C142: 10n, Capacitor_SMD:C_0402_1005Metric, F.Cu at (-106.9, 175.0)
- added C143: 10n, Capacitor_SMD:C_0402_1005Metric, F.Cu at (-106.9, 176.9)
- added C20: 22u, Capacitor_SMD:C_0805_2012Metric, F.Cu at (-77.6, 171.0)
- added C21: 22u, Capacitor_SMD:C_0805_2012Metric, F.Cu at (-56.9, 134.3)
- added C27: 22u, Capacitor_SMD:C_0805_2012Metric, F.Cu at (-56.9, 137.6)
- added C28: 22u, Capacitor_SMD:C_0805_2012Metric, F.Cu at (-56.9, 141.0)
- added C91: 1u, Capacitor_SMD:C_0805_2012Metric, F.Cu at (-12.2, 103.8)
- added C96: 22u, Capacitor_SMD:C_1206_3216Metric, F.Cu at (-103.9, 207.0)
- added C97: 22u, Capacitor_SMD:C_1206_3216Metric, F.Cu at (-103.9, 210.4)
- added J10: Conn_01x02, Connector_JST:JST_GH_BM02B-GHS-TBT_1x02-1MP_P1.25mm_Vertical, F.Cu at (-56.3, 180.3)
- added J15: Bus_M.2_Socket_M, M.2 M Key socket:M.2 M Key socket, B.Cu at (227.6, 105.4)
- added J16: Bus_M.2_Socket_M, M.2 M Key socket:M.2 M Key socket WN HOLES, F.Cu at (227.6, 105.4)
- added J17: Bus_M.2_Socket_M, M.2 M Key socket:M.2 M Key socket WN HOLES, F.Cu at (227.6, 81.3)
- added J18: 10029364-001LF, 87713-1001:87713-1001, F.Cu at (312.7, 80.6)
- added J19: 10029364-001LF, 87713-1001:87713-1001, F.Cu at (312.7, 124.3)
- added Q10: NPN, MMBT3904:P200_SOT-23, F.Cu at (-98.5, 163.3)
- added Q17: NPN, MMBT3904:P200_SOT-23, F.Cu at (-98.5, 167.8)
- added Q2: NPN, MMBT3904:P200_SOT-23, F.Cu at (-99.8, 206.5)
- added R47: 100K, Resistor_SMD:R_0603_1608Metric, F.Cu at (-94.2, 206.6)
- added R65: 100K, Resistor_SMD:R_0603_1608Metric, F.Cu at (-97.8, 172.3)
- added R77: 100K, Resistor_SMD:R_0603_1608Metric, F.Cu at (-97.8, 174.8)
- added U2: TPD4EUSB30, Package_SON:USON-10_2.5x1.0mm_P0.5mm, F.Cu at (235.0, 221.3)
- added U3: TPD4EUSB30, Package_SON:USON-10_2.5x1.0mm_P0.5mm, F.Cu at (229.2, 221.3)
- BT1, C10, C11, C4, C5, C6, C7, C8, C9, D4: moved to B.Cu
- C35: renamed from C31; moved to B.Cu
- C58: renamed from C54; footprint Capacitor_SMD:C_0603_1608Metric -> Capacitor_SMD:C_0402_1005Metric; moved to B.Cu
- C59: renamed from C55; footprint Capacitor_SMD:C_0603_1608Metric -> Capacitor_SMD:C_0402_1005Metric; moved to B.Cu
- C60: renamed from C56; footprint Capacitor_SMD:C_0603_1608Metric -> Capacitor_SMD:C_0402_1005Metric; moved to B.Cu
- C61: renamed from C57; footprint Capacitor_SMD:C_0603_1608Metric -> Capacitor_SMD:C_0402_1005Metric; moved to B.Cu
- C62: renamed from C58; footprint Capacitor_SMD:C_0603_1608Metric -> Capacitor_SMD:C_0402_1005Metric; moved to B.Cu
- C63: renamed from C59; footprint Capacitor_SMD:C_0603_1608Metric -> Capacitor_SMD:C_0402_1005Metric; moved to B.Cu
- C69: renamed from C65; footprint Capacitor_SMD:C_0603_1608Metric -> Capacitor_SMD:C_0402_1005Metric; moved to B.Cu
- C70: renamed from C66; footprint Capacitor_SMD:C_0603_1608Metric -> Capacitor_SMD:C_0402_1005Metric; moved to B.Cu
- C71: renamed from C67; footprint Capacitor_SMD:C_0603_1608Metric -> Capacitor_SMD:C_0402_1005Metric; moved to B.Cu
- C72: renamed from C68; footprint Capacitor_SMD:C_0603_1608Metric -> Capacitor_SMD:C_0402_1005Metric; moved to B.Cu
- C73: renamed from C69; footprint Capacitor_SMD:C_0603_1608Metric -> Capacitor_SMD:C_0402_1005Metric; moved to B.Cu
- C74: renamed from C70; footprint Capacitor_SMD:C_0603_1608Metric -> Capacitor_SMD:C_0402_1005Metric; moved to B.Cu
- C82: renamed from C78; footprint Capacitor_SMD:C_0603_1608Metric -> Capacitor_SMD:C_0402_1005Metric
- C83: renamed from C79; footprint Capacitor_SMD:C_0603_1608Metric -> Capacitor_SMD:C_0402_1005Metric
- C84: renamed from C80; footprint Capacitor_SMD:C_0603_1608Metric -> Capacitor_SMD:C_0402_1005Metric
- C85: renamed from C81; footprint Capacitor_SMD:C_0603_1608Metric -> Capacitor_SMD:C_0402_1005Metric
- C86: renamed from C82; footprint Capacitor_SMD:C_0603_1608Metric -> Capacitor_SMD:C_0402_1005Metric
- C87: renamed from C83; footprint Capacitor_SMD:C_0603_1608Metric -> Capacitor_SMD:C_0402_1005Metric
- IC1: footprint TPS65251-1RHAR:QFN50P600X600X100-41N-D -> Package_DFN_QFN:VQFN-40-1EP_6x6mm_P0.5mm_EP3.5x3.5mm_ThermalVias
- J14: value JST_SHBM04B-SRSS-TB -> Bus_M.2_Socket_M; footprint Connector_JST:JST_SH_BM04B-SRSS-TB_1x04-1MP_P1.00mm_Vertical -> M.2 M Key socket:M.2 M Key socket; moved to B.Cu
- J2: renamed from J3; moved to B.Cu
- J20, J21: value 47018-2000 -> 10029364-001LF; footprint 47018-2000:MOLEX_47018-2000 -> 87713-1001:87713-1001
- J4: renamed from J6; moved to B.Cu
- J6: renamed from J8; moved to B.Cu
- U10, U12: footprint Package_DFN_QFN:QFN-64-1EP_8x8mm_P0.4mm_EP6.5x6.5mm -> Package_DFN_QFN:QFN-64-1EP_8x8mm_P0.4mm_EP6.5x6.5mm_ThermalVias
- U8: footprint Package_DFN_QFN:QFN-64-1EP_9x9mm_P0.5mm_EP5.2x5.2mm -> Package_DFN_QFN:QFN-64-1EP_9x9mm_P0.5mm_EP5.2x5.2mm_ThermalVias
- moved J4 471.8 mm to (312.4, 222.8), turned to -90 degrees
- moved J2 459.0 mm to (310.8, 207.4), turned to -90 degrees
- moved J8 456.0 mm to (302.1, 239.9)
- moved BT1 454.8 mm to (304.9, 161.1), turned to -90 degrees
- moved J5 437.6 mm to (288.4, 234.7)
- moved J6 435.9 mm to (312.5, 182.2), turned to -90 degrees
- moved J21 429.0 mm to (312.8, 211.6), turned to 90 degrees
- moved J1 424.4 mm to (251.6, 241.3)
- moved J20 418.3 mm to (312.8, 167.9), turned to 90 degrees
- moved C2 411.0 mm to (242.7, 233.3), turned to 180 degrees
- moved C1 409.6 mm to (242.7, 228.0)
- moved Module1 408.1 mm to (222.6, 211.9)
- moved U1 401.4 mm to (245.2, 230.7)
- moved H2 399.1 mm to (312.1, 240.0)
- moved J3 399.0 mm to (226.8, 224.8)
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- renumbered TP3 to +12V1, TP4 to +5V1, C92 to C100, C93 to C101, C94 to C102, C98 to C103, C105 to C104, C104 to C105, C103 to C106, C99 to C107, C106 to C108, C107 to C109, C108 to C110, C109 to C111, C100 to C112, C101 to C113, C102 to C114, C110 to C115, C111 to C116, C112 to C117, C113 to C118, C114 to C119, C118 to C119, C119 to C120, C115 to C120, C116 to C121, C117 to C122, C122 to C123, C120 to C123, C121 to C124, C123 to C124, C124 to C125, C125 to C126, C126 to C127, C128 to C129, C129 to C130, C130 to C131, C131 to C132, C127 to C132, C133 to C134, C132 to C134, C134 to C135, C135 to C136, C136 to C137, C137 to C138, C138 to C139, C139 to C144, C140 to C145, C141 to C146, C142 to C147, C143 to C148, C144 to C149, C145 to C150, C146 to C151, C147 to C152, C148 to C153, C149 to C154, C150 to C155, C151 to C156, C152 to C157, C153 to C158, C20 to C22, C21 to C23, C22 to C24, C23 to C25, C24 to C26, C25 to C29, C26 to C30, C27 to C31, C28 to C32, C29 to C33, C30 to C34, C32 to C36, C33 to C37, C34 to C38, C35 to C39, C36 to C40, C37 to C41, C38 to C42, C39 to C43, C40 to C44, C41 to C45, C42 to C46, C43 to C47, C44 to C48, C45 to C49, C46 to C50, C47 to C51, C48 to C52, C49 to C53, C50 to C54, C51 to C55, C52 to C56, C53 to C57, C60 to C64, C61 to C65, C62 to C66, C63 to C67, C64 to C68, C71 to C75, C72 to C76, C73 to C77, C74 to C78, C75 to C79, C76 to C80, C77 to C81, C84 to C88, C85 to C89, C86 to C90, C87 to C92, C88 to C93, C89 to C94, C90 to C95, C95 to C96, C96 to C98, C97 to C98, C91 to C99, TP5 to GND1, J2 to J1, J12 to J11, J13 to J12, J15 to J13, J24 to J22, J5 to J3, J7 to J5, J9 to J7, J10 to J8, J11 to J9, Q16 to Q15, Q17 to Q16, Q9 to Q8, Q8 to Q9, R3 to R1, R12 to R10, R13 to R11, R14 to R12, R15 to R13, R16 to R14, R17 to R15, R18 to R16, R19 to R17, R20 to R18, R21 to R19, R4 to R2, R22 to R20, R23 to R21, R24 to R22, R25 to R23, R26 to R24, R27 to R25, R28 to R26, R29 to R27, R30 to R28, R31 to R29, R5 to R3, R32 to R30, R33 to R31, R34 to R32, R35 to R33, R36 to R34, R37 to R35, R38 to R36, R39 to R37, R40 to R38, R41 to R39, R6 to R4, R42 to R40, R43 to R41, R44 to R42, R45 to R43, R46 to R44, R47 to R45, R48 to R46, R50 to R48, R51 to R49, R7 to R5, R52 to R50, R53 to R51, R54 to R52, R55 to R53, R57 to R54, R58 to R55, R59 to R56, R60 to R57, R61 to R58, R56 to R59, R8 to R6, R62 to R60, R63 to R61, R64 to R62, R65 to R63, R66 to R64, R68 to R66, R69 to R67, R70 to R68, R71 to R69, R9 to R7, R72 to R70, R73 to R71, R75 to R72, R76 to R73, R77 to R74, R78 to R75, R79 to R76, R80 to R78, R81 to R79, R10 to R8, R82 to R80, R83 to R81, R84 to R82, R85 to R83, R86 to R84, R11 to R9, TP6 to TP3, TP7 to TP4, TP8 to TP5, TP9 to TP6, TP10 to TP7, TP11 to TP8, TP12 to TP9
Connections:
- +12V1 pad 1: Net-(F1-Pad1) -> /Project Architecture/Input/+12V
- +5V1 pad 1: Net-(F2-Pad1) -> /Project Architecture/Input/+5V
- C100 pad 2: Net-(C92-Pad2) -> Net-(C100-Pad2)
- C101 pad 2: Net-(C93-Pad2) -> Net-(C101-Pad2)
- C102 pad 2: Net-(C94-Pad2) -> Net-(C102-Pad2)
- C105 pad 1: +5V-HDD1 -> gnd
- C105 pad 2: gnd -> +5V-HDD1
- C107 pad 2: Net-(C99-Pad2) -> Net-(C107-Pad2)
- C112 pad 2: Net-(C100-Pad2) -> Net-(C112-Pad2)
- C113 pad 2: Net-(C101-Pad2) -> Net-(C113-Pad2)
- C114 pad 2: Net-(C102-Pad2) -> Net-(C114-Pad2)
- C12 pad 1: /Project Architecture/Input/+5V S1 -> /Project Architecture/Input/+5V
- C13 pad 1: /Project Architecture/Input/+5V S1 -> /Project Architecture/Input/+5V
- C14 pad 1: /Project Architecture/Input/+5V S1 -> /Project Architecture/Input/+5V
- C15 pad 1: /Project Architecture/Input/+5V S1 -> /Project Architecture/Input/+5V
- C16 pad 1: /Project Architecture/Input/+5V S1 -> /Project Architecture/Input/+5V
- C17 pad 1: /Project Architecture/Input/+5V S1 -> /Project Architecture/Input/+5V
- C18 pad 1: /Project Architecture/Input/+5V S1 -> /Project Architecture/Input/+5V
- C19 pad 1: /Project Architecture/Input/+5V S1 -> /Project Architecture/Input/+5V
- C77 pad 1: Net-(IC3-PGND2_1) -> gnd
- C77 pad 2: /Project Architecture/M.2 Drives/+5V S1 -> /Project Architecture/M.2 Drives/EN
- C78 pad 1: Net-(IC3-PGND2_1) -> gnd
- C78 pad 2: /Project Architecture/M.2 Drives/+5V S1 -> /Project Architecture/M.2 Drives/EN
- C80 pad 1: /Project Architecture/M.2 Drives/+5V S1 -> /Project Architecture/M.2 Drives/EN
- C80 pad 2: Net-(IC3-PGND1_1) -> gnd
- C81 pad 1: /Project Architecture/M.2 Drives/+5V S1 -> /Project Architecture/M.2 Drives/EN
- C81 pad 2: Net-(IC3-PGND1_1) -> gnd
- C99 pad 2: Net-(C91-Pad2) -> Net-(C99-Pad2)
- D5 pad 2: /Project Architecture/Input/+5V S1 -> /Project Architecture/Input/+5V
- F1 pad 1: Net-(F1-Pad1) -> /Project Architecture/Input/+12V
- F2 pad 1: Net-(F2-Pad1) -> /Project Architecture/Input/+5V
- F2 pad 2: /Project Architecture/Input/+5V S1 -> /Project Architecture/Input/+5V
- IC3 pad 1: Net-(IC3-PGND2_1) -> gnd
- IC3 pad 14: /Project Architecture/M.2 Drives/+5V S1 -> /Project Architecture/M.2 Drives/EN
- IC3 pad 15: Net-(IC3-PGND1_1) -> gnd
- IC3 pad 2: /Project Architecture/M.2 Drives/+5V S1 -> /Project Architecture/M.2 Drives/EN
- J13 pad 2: Net-(F2-Pad1) -> /Project Architecture/Input/+5V
- J13 pad 3: Net-(F1-Pad1) -> /Project Architecture/Input/+12V
- J14 pad 1: /Project Architecture/CM5_GPIO/+12V -> gnd
- J14 pad 2: /Project Architecture/CM5_GPIO/PWM_3 -> /Project Architecture/M.2 Drives/FB
- J14 pad 4: unconnected-(J14-Pin_4-Pad4) -> /Project Architecture/M.2 Drives/FB
- Module1 pad 88: /Project Architecture/CM5_GPIO/+1V8 -> unconnected-(Module1A-+1.8v_(Output)-Pad88)
- Module1 pad 90: /Project Architecture/CM5_GPIO/+1V8 -> unconnected-(Module1A-+1.8v_(Output)-Pad90)
- Q9 pad 2: Net-(Q8-B) -> Net-(Q9-B)
- R42 pad 2: Net-(J16-DAS/~{DSS}/~{LED1}) (its old number) -> Net-(J14-DAS/~{DSS}/~{LED1})
- R59 pad 2: Net-(Q8-B) -> Net-(Q9-B)
- U8 pad 2: /Project Architecture/M.2 Drives/gnd{PERST} -> /Project Architecture/M.2 Drives/PERST
Routing:
- net Net-(IC1-SS3): track 0.00 -> 6.67 mm
- net Net-(IC1-RLIM3): track 0.00 -> 4.02 mm
- net Net-(IC1-CMP3): track 0.00 -> 3.95 mm
- net Net-(IC1-BST3): track 0.00 -> 1.57 mm, vias 0 -> 1
- net Net-(C46-Pad1): track 0.00 -> 1.24 mm
- net Net-(IC1-LX3_1): track 0.00 -> 0.78 mm, vias 0 -> 1
Other:
- board outline added: 100 x 193 mm
- board text added: "+12V"
- board text added: "+5V"
- board text added: "12V"
- board text added: "5V"
- board text added: "Battery CR2032"
- board text added: "CHANGE to 0402"
- board text added: "Change two 3 pin"
- board text added: "Compute Module 5"
- board text added: "GND"

Commit message: More pcbing
Parts:
- removed C28: 22u, Capacitor_SMD:C_0805_2012Metric
- removed TP9: TestPoint, TestPoint:TestPoint_Pad_1.0x1.0mm
- added C94: 47u, Capacitor_SMD:C_0805_2012Metric, F.Cu at (278.8, 97.9)
- C20, C34, C38, C39, C40, C41, C46, C47, C50, C51, IC1, L2, R20, R22, R26, R27: moved to B.Cu
- C35, J15: moved to F.Cu
- C49, C53: footprint Capacitor_SMD:C_0805_2012Metric -> Capacitor_SMD:C_0402_1005Metric
- C52: footprint Capacitor_SMD:C_0603_1608Metric -> Capacitor_SMD:C_0402_1005Metric
- J16: footprint M.2 M Key socket:M.2 M Key socket WN HOLES -> M.2 M Key socket:M.2 M Key socket
- J17: footprint M.2 M Key socket:M.2 M Key socket WN HOLES -> M.2 M Key socket:M.2 M Key socket; moved to B.Cu
- J18, J19, J20, J21: value 10029364-001LF -> 0877131001
- R18, R19, R23, R24, R25: footprint Resistor_SMD:R_0603_1608Metric -> Resistor_SMD:R_0402_1005Metric; moved to B.Cu
- R28: footprint Resistor_SMD:R_0603_1608Metric -> Capacitor_SMD:C_0402_1005Metric
- R35: footprint Resistor_SMD:R_0603_1608Metric -> Resistor_SMD:R_0402_1005Metric
- moved H5 349.3 mm to (-50.8, 0.00)
- moved C77 315.6 mm to (289.1, 88.8), turned to 90 degrees
- moved C91 314.7 mm to (287.9, 94.1), turned to 90 degrees
- moved C92 314.6 mm to (287.9, 97.9), turned to -90 degrees
- moved C78 309.2 mm to (287.0, 88.7), turned to 90 degrees
- moved C93 305.3 mm to (278.8, 94.2), turned to 90 degrees
- moved C79 304.1 mm to (286.7, 86.2), turned to 90 degrees
- moved C81 304.0 mm to (277.2, 88.5), turned to -90 degrees
- moved L5 303.9 mm to (283.3, 94.1), turned to -90 degrees
- moved C80 301.7 mm to (279.5, 88.3), turned to -90 degrees
- moved R35 297.5 mm to (279.3, 84.7), turned to 180 degrees
- moved IC3 296.9 mm to (283.3, 87.0), turned to 180 degrees
- moved C90 296.3 mm to (283.3, 82.4), turned to 180 degrees
- moved C44 296.3 mm to (232.5, 59.6), turned to -90 degrees
- moved J7 294.1 mm to (-68.6, 199.4)
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- renumbered C99 to C100, C100 to C101, C101 to C102, C102 to C103, C103 to C104, C104 to C105, C105 to C106, C106 to C107, C107 to C108, C108 to C109, C109 to C110, C110 to C111, C111 to C112, C112 to C113, C113 to C114, C114 to C115, C115 to C116, C116 to C117, C117 to C118, C118 to C119, C119 to C120, C120 to C121, C121 to C122, C122 to C123, C123 to C124, C124 to C125, C125 to C126, C126 to C127, C127 to C128, C128 to C129, C129 to C130, C130 to C131, C131 to C132, C132 to C133, C133 to C134, C134 to C135, C135 to C136, C136 to C137, C137 to C138, C138 to C139, C139 to C140, C140 to C141, C141 to C142, C142 to C143, C143 to C144, C144 to C145, C145 to C146, C146 to C147, C147 to C148, C148 to C149, C149 to C150, C150 to C151, C151 to C152, C152 to C153, C153 to C154, C154 to C155, C155 to C156, C156 to C157, C157 to C158, C158 to C159, C91 to C90, C92 to C91, C93 to C92, C90 to C93, C94 to C95, C95 to C96, C96 to C97, C97 to C98, C98 to C99
Connections:
- net /Project Architecture/M.2 Drives/EN renamed /Project Architecture/M.2 Drives/+5V S1
- net /Project Architecture/M.2 Drives/FB renamed /Project Architecture/M.2 Drives/+3V3 M.2
- net Net-(U8-TXN_3) renamed /Project Architecture/M.2 Drives/TX_N_3
- net Net-(U8-TXP_3) renamed /Project Architecture/M.2 Drives/TX_P_3
- C100 pad 2: Net-(C99-Pad2) -> Net-(J18-S6)
- C101 pad 2: Net-(C100-Pad2) -> Net-(J18-S5)
- C102 pad 2: Net-(C101-Pad2) -> Net-(J18-S3)
- C103 pad 2: Net-(C102-Pad2) -> Net-(J18-S2)
- C108 pad 2: Net-(C107-Pad2) -> Net-(J19-S6)
- C113 pad 2: Net-(C112-Pad2) -> Net-(J19-S5)
- C114 pad 2: Net-(C113-Pad2) -> Net-(J19-S3)
- C115 pad 2: Net-(C114-Pad2) -> Net-(J19-S2)
- C12 pad 1: /Project Architecture/Input/+5V -> /Project Architecture/Input/+5V S1
- C129 pad 2: Net-(C128-Pad2) -> Net-(J20-S6)
- C13 pad 1: /Project Architecture/Input/+5V -> /Project Architecture/Input/+5V S1
- C130 pad 2: Net-(C129-Pad2) -> Net-(J20-S5)
- C131 pad 2: Net-(C130-Pad2) -> Net-(J20-S3)
- C132 pad 2: Net-(C131-Pad2) -> Net-(J20-S2)
- C14 pad 1: /Project Architecture/Input/+5V -> /Project Architecture/Input/+5V S1
- C141 pad 2: Net-(C140-Pad2) -> Net-(J21-S6)
- C142 pad 2: Net-(C141-Pad2) -> Net-(J21-S5)
- C143 pad 2: Net-(C142-Pad2) -> Net-(J21-S3)
- C144 pad 2: Net-(C143-Pad2) -> Net-(J21-S2)
- C15 pad 1: /Project Architecture/Input/+5V -> /Project Architecture/Input/+5V S1
- C16 pad 1: /Project Architecture/Input/+5V -> /Project Architecture/Input/+5V S1
- C17 pad 1: /Project Architecture/Input/+5V -> /Project Architecture/Input/+5V S1
- C18 pad 1: /Project Architecture/Input/+5V -> /Project Architecture/Input/+5V S1
- C19 pad 1: /Project Architecture/Input/+5V -> /Project Architecture/Input/+5V S1
- C43 pad 1: /Project Architecture/Power/+12V -> /Project Architecture/Power/SUP
- C44 pad 1: /Project Architecture/Power/+12V -> /Project Architecture/Power/SUP
- C45 pad 1: /Project Architecture/Power/+12V -> /Project Architecture/Power/SUP
- D5 pad 2: /Project Architecture/Input/+5V -> /Project Architecture/Input/+5V S1
- F2 pad 2: /Project Architecture/Input/+5V -> /Project Architecture/Input/+5V S1
- IC2 pad 11: /Project Architecture/Power/+12V -> /Project Architecture/Power/SUP
- IC3 pad 16: Net-(IC3-SW) -> /Project Architecture/M.2 Drives/BOOT
- J15 pad 53: /Project Architecture/M.2 Drives/PCIe_CLK_N_4 -> /Project Architecture/M.2 Drives/PCIe_CLK_N_3
- J15 pad 55: /Project Architecture/M.2 Drives/PCIe_CLK_P_4 -> /Project Architecture/M.2 Drives/PCIe_CLK_P_3
- J18 pad 1: (no net) -> gnd
- J18 pad 10: (no net) -> unconnected-(J18-P3-Pad10)
- J18 pad 11: (no net) -> gnd
- J18 pad 12: (no net) -> Net-(J18-P5)
- J18 pad 13: (no net) -> gnd
- J18 pad 14: (no net) -> +5V-HDD0
- J18 pad 15: (no net) -> +5V-HDD0
- J18 pad 16: (no net) -> +5V-HDD0
- J18 pad 17: (no net) -> gnd
- J18 pad 18: (no net) -> gnd
- J18 pad 19: (no net) -> gnd
- J18 pad 2: (no net) -> Net-(J18-S2)
- J18 pad 20: (no net) -> +12V-HDD0
- J18 pad 21: (no net) -> +12V-HDD0
- J18 pad 22: (no net) -> +12V-HDD0
- J18 pad 3: (no net) -> Net-(J18-S3)
- J18 pad 4: (no net) -> gnd
- J18 pad 5: (no net) -> Net-(J18-S5)
- J18 pad 6: (no net) -> Net-(J18-S6)
- J18 pad 7: (no net) -> gnd
- J18 pad 8: (no net) -> unconnected-(J18-P1-Pad8)
- J18 pad 9: (no net) -> unconnected-(J18-P2-Pad9)
- J19 pad 1: (no net) -> gnd
- J19 pad 10: (no net) -> unconnected-(J19-P3-Pad10)
- J19 pad 11: (no net) -> gnd
- J19 pad 12: (no net) -> Net-(J19-P5)
- J19 pad 13: (no net) -> gnd
- J19 pad 14: (no net) -> +5V-HDD1
- J19 pad 15: (no net) -> +5V-HDD1
- J19 pad 16: (no net) -> +5V-HDD1
- J19 pad 17: (no net) -> gnd
- J19 pad 18: (no net) -> gnd
- J19 pad 19: (no net) -> gnd
- J19 pad 2: (no net) -> Net-(J19-S2)
- J19 pad 20: (no net) -> +12V-HDD1
- J19 pad 21: (no net) -> +12V-HDD1
- J19 pad 22: (no net) -> +12V-HDD1
- J19 pad 3: (no net) -> Net-(J19-S3)
- J19 pad 4: (no net) -> gnd
- J19 pad 5: (no net) -> Net-(J19-S5)
- J19 pad 6: (no net) -> Net-(J19-S6)
- J19 pad 7: (no net) -> gnd
- J19 pad 8: (no net) -> unconnected-(J19-P1-Pad8)
- J19 pad 9: (no net) -> unconnected-(J19-P2-Pad9)
- J20 pad 1: (no net) -> gnd
- J20 pad 10: (no net) -> unconnected-(J20-P3-Pad10)
- J20 pad 11: (no net) -> gnd
- J20 pad 12: (no net) -> Net-(J20-P5)
- J20 pad 13: (no net) -> gnd
- J20 pad 14: (no net) -> +5V-HDD2
- J20 pad 15: (no net) -> +5V-HDD2
- J20 pad 16: (no net) -> +5V-HDD2
- J20 pad 17: (no net) -> gnd
- J20 pad 18: (no net) -> gnd
- J20 pad 19: (no net) -> gnd
- J20 pad 2: (no net) -> Net-(J20-S2)
- J20 pad 20: (no net) -> +12V-HDD2
- J20 pad 21: (no net) -> +12V-HDD2
- J20 pad 22: (no net) -> +12V-HDD2
- J20 pad 3: (no net) -> Net-(J20-S3)
- J20 pad 4: (no net) -> gnd
- J20 pad 5: (no net) -> Net-(J20-S5)
- J20 pad 6: (no net) -> Net-(J20-S6)
- J20 pad 7: (no net) -> gnd
- J20 pad 8: (no net) -> unconnected-(J20-P1-Pad8)
- J20 pad 9: (no net) -> unconnected-(J20-P2-Pad9)
- J21 pad 1: (no net) -> gnd
- J21 pad 10: (no net) -> unconnected-(J21-P3-Pad10)
- J21 pad 11: (no net) -> gnd
- J21 pad 12: (no net) -> Net-(J21-P5)
- J21 pad 13: (no net) -> gnd
- J21 pad 14: (no net) -> +5V-HDD3
- J21 pad 15: (no net) -> +5V-HDD3
- J21 pad 16: (no net) -> +5V-HDD3
- J21 pad 17: (no net) -> gnd
- J21 pad 18: (no net) -> gnd
- J21 pad 19: (no net) -> gnd
- J21 pad 2: (no net) -> Net-(J21-S2)
- J21 pad 20: (no net) -> +12V-HDD3
- J21 pad 21: (no net) -> +12V-HDD3
- J21 pad 22: (no net) -> +12V-HDD3
- J21 pad 3: (no net) -> Net-(J21-S3)
- J21 pad 4: (no net) -> gnd
- J21 pad 5: (no net) -> Net-(J21-S5)
- J21 pad 6: (no net) -> Net-(J21-S6)
- J21 pad 7: (no net) -> gnd
- J21 pad 8: (no net) -> unconnected-(J21-P1-Pad8)
- J21 pad 9: (no net) -> unconnected-(J21-P2-Pad9)
- L5 pad 1: Net-(IC3-SW) -> /Project Architecture/M.2 Drives/BOOT
- Q10 pad 2: Net-(Q10-B) -> Net-(J20-P5)
- Q17 pad 2: Net-(Q17-B) -> Net-(J21-P5)
- Q2 pad 2: Net-(Q2-B) -> Net-(J18-P5)
- Q9 pad 2: Net-(Q9-B) -> Net-(J19-P5)
- R47 pad 1: Net-(Q2-B) -> Net-(J18-P5)
- R59 pad 2: Net-(Q9-B) -> Net-(J19-P5)
- R65 pad 1: Net-(Q10-B) -> Net-(J20-P5)
- R77 pad 1: Net-(Q17-B) -> Net-(J21-P5)
Routing:
- net /Project Architecture/M.2 Drives/+3V3 M.2: track 0.00 -> 27.6 mm, vias 0 -> 10
- net /Project Architecture/Power/+5V S2: track 0.00 -> 20.5 mm, vias 0 -> 2
- net /Project Architecture/Power/FB1: track 0.00 -> 8.08 mm
- net /Project Architecture/Power/FB3: track 0.00 -> 7.70 mm
- net Net-(IC1-SS1): track 0.00 -> 7.62 mm
- net /Project Architecture/M.2 Drives/VCC: track 0.00 -> 4.43 mm
- net Net-(IC2-COMP): track 0.00 -> 3.54 mm
- net Net-(IC1-RLIM1): track 0.00 -> 3.31 mm, vias 0 -> 1
- net Net-(IC1-CMP1): track 0.00 -> 3.03 mm
- net Net-(IC2-BIAS): track 0.00 -> 2.97 mm
- net Net-(IC2-FOSC): track 0.00 -> 2.80 mm
- net Net-(IC2-~{RESET}): track 0.00 -> 2.74 mm, vias 0 -> 1
- net /Project Architecture/M.2 Drives/TX_P_3: track 0.00 -> 1.74 mm
- net Net-(IC1-BST3): track 1.57 -> 0.00 mm, vias 1 -> 0
- net /Project Architecture/M.2 Drives/TX_N_3: track 0.00 -> 1.30 mm
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Other:
- board text removed: "+12V"
- board text removed: "+5V"

Commit message: More pcb arangment, verticle ports
Parts:
- removed C157, C158: 100n, Capacitor_SMD:C_0603_1608Metric
- removed the C98 at (-66.3, 50.9)
- removed the R47 at (-94.2, 206.6)
- removed the R82 at (-23.7, 23.1)
- removed the R83 at (-23.7, 25.6)
- removed the TP4 at (-35.6, 139.6)
- removed the U11 at (-59.4, 117.6)
- removed the U2 at (-139.9, 120.6)
- removed the U3 at (-137.1, 120.6)
- removed the U9 at (-50.1, 59.5)
- added C160: 0u01, Capacitor_SMD:C_0402_1005Metric, F.Cu at (278.9, 203.7)
- added C28: 22u, Capacitor_SMD:C_0805_2012Metric, B.Cu at (278.5, 77.4)
- added J23: USB_A, 482040001:CONN_48204-0001_MOL, F.Cu at (265.3, 225.0)
- added JP3: 3P_JUMPER, Connector_PinHeader_2.54mm:PinHeader_1x03_P2.54mm_Vertical, F.Cu at (-52.7, 58.4)
- added R12: 10K, Resistor_SMD:R_0603_1608Metric, B.Cu at (266.6, 87.3)
- added R65: 100K, Resistor_SMD:R_0603_1608Metric, F.Cu at (-48.4, 57.4)
- added R87: 12K, Resistor_SMD:R_0603_1608Metric, F.Cu at (275.5, 205.6)
- added U10: W25X20CLUXIG_TR, W25X20CLUXIG_TR:SON50P300X200X60-9N, F.Cu at (-48.9, 112.7)
- added U12: W25X20CLUXIG_TR, W25X20CLUXIG_TR:SON50P300X200X60-9N, F.Cu at (-48.9, 107.1)
- C109, C110, C111, C112, C116, C117, C120, C121, C123: footprint Capacitor_SMD:C_0603_1608Metric -> Capacitor_SMD:C_0402_1005Metric
- C118, C119, C122: footprint Capacitor_SMD:C_0805_2012Metric -> Capacitor_SMD:C_0402_1005Metric
- C159: value 0u01 -> 100n; footprint Capacitor_SMD:C_0402_1005Metric -> Capacitor_SMD:C_0603_1608Metric
- C21, C22, C26, C27, C30, C31, C32, C37, L1, L3, R48, R49: moved to B.Cu
- C23, C29, C99: footprint Capacitor_SMD:C_0805_2012Metric -> Capacitor_SMD:C_0603_1608Metric; moved to B.Cu
- J1: footprint 10029449-111RLF:AMPHENOL_10029449-111RLF -> G45A19071083HR:AMPHENOL_G45A19071083HR
- J14, J17: footprint M.2 M Key socket:M.2 M Key socket -> 2199119-5:21991195 no holes
- J15, J16: footprint M.2 M Key socket:M.2 M Key socket -> 2199119-5:21991195
- J22: value USB_A_Stacked -> USB_A; footprint Connector_USB:USB_A_Wuerth_61400826021_Horizontal_Stacked -> 482040001:CONN_48204-0001_MOL
- Q2: value NPN -> MMBT3904; footprint MMBT3904:P200_SOT-23 -> Package_TO_SOT_SMD:SOT-23; moved to B.Cu
- Q3, Q5: value PMOS -> AOSS21311C; footprint AOSS21311C:SOT95P237X117-3N -> Package_TO_SOT_SMD:SOT-23-3; moved to B.Cu
- Q4: value NPN -> AOSS21311C; footprint MMBT3904:P200_SOT-23 -> Package_TO_SOT_SMD:SOT-23; moved to B.Cu
- Q6, Q8: value PMOS -> AOSS21311C; footprint AOSS21311C:SOT95P237X117-3N -> Package_TO_SOT_SMD:SOT-23-3
- Q7, Q9: value NPN -> MMBT3904
- R11: footprint Resistor_SMD:R_0603_1608Metric -> Resistor_SMD:R_0402_1005Metric; moved to B.Cu
- R13: renamed from R12; footprint Resistor_SMD:R_0603_1608Metric -> Resistor_SMD:R_0402_1005Metric; moved to B.Cu
- R14: renamed from R13; footprint Resistor_SMD:R_0603_1608Metric -> Resistor_SMD:R_0402_1005Metric; moved to B.Cu
- R15: renamed from R14; footprint Resistor_SMD:R_0603_1608Metric -> Resistor_SMD:R_0402_1005Metric; moved to B.Cu
- R50: renamed from R49; moved to B.Cu
- R51: renamed from R50; footprint Resistor_SMD:R_0603_1608Metric -> Resistor_SMD:R_0402_1005Metric; moved to B.Cu
- R53: renamed from R52; footprint Resistor_SMD:R_0603_1608Metric -> Resistor_SMD:R_0402_1005Metric; moved to B.Cu
- R56: renamed from R55; moved to B.Cu
- R58: renamed from R57; moved to B.Cu
- R84: value 12K -> 1K
- moved C110 449.1 mm to (329.8, 190.4)
- moved R48 446.8 mm to (334.6, 184.9), turned to 180 degrees
- moved R53 445.8 mm to (332.6, 190.4)
- moved R51 444.7 mm to (332.6, 189.5), turned to 180 degrees
- moved R56 444.2 mm to (328.2, 208.6), turned to 180 degrees
- moved C104 444.0 mm to (346.4, 200.6)
- moved Q6 444.0 mm to (336.8, 207.6)
- moved Q7 444.0 mm to (340.6, 206.2)
- moved Q8 444.0 mm to (336.8, 212.1)
- moved R54 444.0 mm to (328.3, 199.8)
- moved R55 444.0 mm to (328.3, 204.9)
- moved R58 443.8 mm to (330.4, 206.0), turned to 180 degrees
- moved Q2 434.7 mm to (334.5, 187.7), turned to -90 degrees
- moved R49 430.5 mm to (302.4, 223.7), turned to -90 degrees
- moved R50 430.3 mm to (304.7, 223.0)
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- renumbered JP3 to JP4, JP4 to JP5, R15 to R16, R16 to R17, R17 to R18, R18 to R19, R19 to R20, R20 to R21, R21 to R22, R22 to R23, R23 to R24, R24 to R25, R25 to R26, R26 to R27, R27 to R28, R28 to R29, R29 to R30, R30 to R31, R31 to R32, R32 to R33, R33 to R34, R34 to R35, R35 to R36, R36 to R37, R37 to R38, R38 to R39, R39 to R40, R40 to R41, R41 to R42, R42 to R43, R43 to R44, R44 to R45, R45 to R46, R46 to R47, R51 to R52, R53 to R54, R54 to R55, R56 to R57, R58 to R59, R59 to R60, R60 to R61, R61 to R62, R62 to R63, R63 to R64, R64 to R66, R65 to R67, R66 to R68, R67 to R69, R68 to R70, R69 to R71, R70 to R72, R71 to R73, R72 to R74, R73 to R75, R74 to R76, R75 to R77, R76 to R78, R77 to R79, R78 to R80, R79 to R81, R80 to R82, R81 to R83, TP5 to TP4, TP6 to TP5, TP7 to TP6, TP8 to TP7, U12 to U11, U10 to U9
Connections:
- net /Project Architecture/CM5_High Speed IO/PCIE_CLK_N renamed /Project Architecture/CM5_High Speed IO/PCIe_CLK_N
- net /Project Architecture/CM5_High Speed IO/PCIE_CLK_P renamed /Project Architecture/CM5_High Speed IO/PCIe_CLK_P
- net /Project Architecture/CM5_High Speed IO/PCIE_RX_N renamed /Project Architecture/CM5_High Speed IO/PCIe_RX_N
- net /Project Architecture/CM5_High Speed IO/PCIE_RX_P renamed /Project Architecture/CM5_High Speed IO/PCIe_RX_P
- net /Project Architecture/CM5_High Speed IO/PCIE_TX_N renamed /Project Architecture/CM5_High Speed IO/PCIe_TX_N
- net /Project Architecture/CM5_High Speed IO/PCIE_TX_P renamed /Project Architecture/CM5_High Speed IO/PCIe_TX_P
- net /Project Architecture/Input/+5V S1 renamed +5V S1
- net /Project Architecture/M.2 Drives/PCIE_CLK_N renamed /Project Architecture/M.2 Drives/PCIe_CLK_N
- net /Project Architecture/M.2 Drives/PCIE_CLK_P renamed /Project Architecture/M.2 Drives/PCIe_CLK_P
- net /Project Architecture/M.2 Drives/PCIE_RX_N renamed /Project Architecture/M.2 Drives/PCIe_RX_N
- net /Project Architecture/M.2 Drives/PCIE_RX_P renamed /Project Architecture/M.2 Drives/PCIe_RX_P
- net /Project Architecture/M.2 Drives/PCIE_TX_N renamed /Project Architecture/M.2 Drives/PCIe_TX_N
- net /Project Architecture/M.2 Drives/PCIE_TX_P renamed /Project Architecture/M.2 Drives/PCIe_TX_P
- +12V1 pad 1: /Project Architecture/Input/+12V -> +12V
- C10 pad 1: /Project Architecture/Input/+12V -> +12V
- C11 pad 1: /Project Architecture/Input/+12V -> +12V
- C4 pad 1: /Project Architecture/Input/+12V -> +12V
- C5 pad 1: /Project Architecture/Input/+12V -> +12V
- C6 pad 1: /Project Architecture/Input/+12V -> +12V
- C7 pad 1: /Project Architecture/Input/+12V -> +12V
- C8 pad 1: /Project Architecture/Input/+12V -> +12V
- C9 pad 1: /Project Architecture/Input/+12V -> +12V
- D4 pad 2: /Project Architecture/Input/+12V -> +12V
- F1 pad 1: /Project Architecture/Input/+12V -> +12V
- F1 pad 2: /Project Architecture/Input/+12V -> +12V
- IC4 pad 1: Net-(IC4-USBDM_DN1/PRT_DIS_M1) -> /Project Architecture/Usb Switch/D1-
- IC4 pad 2: Net-(IC4-USBDP_DN1/PRT_DIS_P1) -> /Project Architecture/Usb Switch/D1+
- IC4 pad 3: Net-(IC4-USBDM_DN2/PRT_DIS_M2) -> /Project Architecture/Usb Switch/D2-
- IC4 pad 4: Net-(IC4-USBDP_DN2/PRT_DIS_P2) -> /Project Architecture/Usb Switch/D2+
- J13 pad 3: /Project Architecture/Input/+12V -> +12V
- J22 pad 2: Net-(IC4-USBDM_DN2/PRT_DIS_M2) -> /Project Architecture/Usb Switch/D1-
- J22 pad 3: Net-(IC4-USBDP_DN2/PRT_DIS_P2) -> /Project Architecture/Usb Switch/D1+
- Q13 pad 3: +5V -> +5V S2
- Q16 pad 3: +5V -> +5V S2
- Q5 pad 3: +5V -> +5V S2
- Q8 pad 3: +5V -> +5V S2
- R48 pad 1: Net-(Q4-C) -> Net-(J18-P5)
- R48 pad 2: +12V -> +5V S2
- R49 pad 1: +5V -> Net-(Q4-C)
- R49 pad 2: Net-(Q2-B) -> +12V
- R60 pad 1: +5V -> +5V S2
- R67 pad 2: +5V -> +5V S2
- R79 pad 2: +5V -> +5V S2
- R84 pad 1: gnd -> /Project Architecture/Usb Switch/+3V3
- R84 pad 2: Net-(IC4-RBIAS) -> Net-(IC4-VBUS_DET)
- R9 pad 2: /Project Architecture/Input/+12V -> +12V
- U11 pad 33: /Project Architecture/Sata Drives 2/VCCH -> /Project Architecture/Sata Drives 2/3V3A
- U9 pad 33: /Project Architecture/Sata Drives 1/VCCH -> /Project Architecture/Sata Drives 1/3V3A
- U9 pad 43: /Project Architecture/Sata Drives 1/VCCH -> /Project Architecture/Sata Drives 1/3V3A
Routing:
- net Net-(IC1-PGOOD): track 0.00 -> 17.3 mm, vias 0 -> 2
- net /Project Architecture/Usb Switch/D2+: track 0.00 -> 14.5 mm
- net /Project Architecture/Usb Switch/D2-: track 0.00 -> 13.0 mm
- net /Project Architecture/CM5_GPIO/TRD0_P: track 0.00 -> 12.8 mm
- net /Project Architecture/CM5_GPIO/TRD0_N: track 0.00 -> 12.1 mm
- net /Project Architecture/Usb Switch/D1+: track 0.00 -> 11.6 mm
- net Net-(Q4-C): track 0.00 -> 10.3 mm
- net /Project Architecture/CM5_GPIO/TRD1_N: track 0.00 -> 10.0 mm
- net /Project Architecture/Usb Switch/D1-: track 0.00 -> 9.84 mm
- net /Project Architecture/CM5_GPIO/TRD1_P: track 0.00 -> 9.56 mm
- net Net-(Q3-G): track 0.00 -> 9.53 mm
- net /Project Architecture/CM5_GPIO/TRD2_P: track 0.00 -> 8.94 mm
- net /Project Architecture/CM5_GPIO/TRD2_N: track 0.00 -> 7.69 mm
- net /Project Architecture/Power/FB2: track 0.00 -> 7.09 mm
- net gnd: track 0.00 -> 5.75 mm, vias 1 -> 3
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