File: Electronics/_autosave-CM5 Nas.kicad_pcb (KiCad board)
At the start: 4 copper layers, 352 parts, among them IC1 TPS65251-1RHAR, IC2 MAX20008AFOC_VY+T, IC3 LM61480Q3RPHRQ1, IC4 USB2512B-AEZG, J1 THD-02-R, J10 JST_SHBM04B-SRSS-TB, J11 JST_SHBM04B-SRSS-TB, J12 JST_SHBM04B-SRSS-TB, J13 JST_SHBM04B-SRSS-TB, J14 JST_SHBM04B-SRSS-TB, J15 4DB-P108-03, J2 HDMI_A, J20 47018-2000, J21 47018-2000, J22 47018-2000, J23 47018-2000, J24 USB_A_Stacked, J3 Conn_01x22_Female, J4 THD-20-R, J5 RJ45_RB1-125B8G1A, J6 Conn_01x07, J7 Micro_SD_Card_Det, J8 Conn_01x04, J9 Conn_02x07_Odd_Even, Q1 PMOS, Q10 NPN, Q11 PMOS, Q12 NPN, Q13 PMOS, Q14 PMOS, Q15 NPN, Q16 NPN, Q17 PMOS, Q2 NPN, Q3 PMOS, Q4 NPN, Q5 PMOS, Q6 PMOS, Q7 NPN, Q8 NPN, Q9 PMOS, SW1 Right angle Tact button, U1 RT9742SNGV, U10 JMS561, U11 W25X40CLSN, U12 JMS561, U2 TPD4EUSB30, U3 TPD4EUSB30, U4 74LVC1G07SE-7, U5 RT9742GGJ5, U6 AMS1117-3.3, U7 ASEK-32.768KHZ-L-R-T, U8 ASM1184, U9 W25X40CLSN, Y1 30MHz, Y2 30MHz, Y3 30MHz

Commit message: Sata Port Changed
Parts:
- added C87: 1u, Capacitor_SMD:C_0805_2012Metric, F.Cu at (-12.2, 103.8)
- added J16: Bus_M.2_Socket_M, M.2 M Key socket:M.2 M Key socket, F.Cu at (58.1, 134.6)
- added J17: Bus_M.2_Socket_M, M.2 M Key socket:M.2 M Key socket, F.Cu at (58.1, 110.5)
- added J18: Bus_M.2_Socket_M, M.2 M Key socket:M.2 M Key socket, F.Cu at (58.1, 86.4)
- added J19: Bus_M.2_Socket_M, M.2 M Key socket:M.2 M Key socket, F.Cu at (58.1, 62.3)
- moved J7 285.9 mm to (140.9, 194.8)
- moved J23 256.5 mm to (168.0, 113.0), turned to 90 degrees
- moved J22 256.0 mm to (168.1, 71.0), turned to 90 degrees
- moved J5 251.4 mm to (84.4, 185.0)
- moved J2 250.7 mm to (63.5, 201.4)
- moved J24 229.3 mm to (113.3, 189.3)
- renumbered C99 to C100, C100 to C101, C101 to C102, C102 to C103, C103 to C104, C104 to C105, C105 to C106, C106 to C107, C107 to C108, C108 to C109, C109 to C110, C110 to C111, C111 to C112, C112 to C113, C113 to C114, C114 to C115, C115 to C116, C116 to C117, C117 to C118, C118 to C119, C119 to C120, C120 to C121, C121 to C122, C122 to C123, C123 to C124, C124 to C125, C125 to C126, C126 to C127, C127 to C128, C128 to C129, C129 to C130, C130 to C131, C131 to C132, C132 to C133, C133 to C134, C134 to C135, C135 to C136, C136 to C137, C137 to C138, C138 to C139, C139 to C140, C140 to C141, C141 to C142, C142 to C143, C143 to C144, C144 to C145, C145 to C146, C146 to C147, C147 to C148, C148 to C149, C149 to C150, C150 to C151, C151 to C152, C152 to C153, C153 to C154, C87 to C88, C88 to C89, C89 to C90, C90 to C91, C91 to C92, C92 to C93, C93 to C94, C94 to C95, C95 to C96, C96 to C97, C97 to C98, C98 to C99
Connections:
- C73 pad 1: Net-(IC3-PGND2_1) -> gnd
- C73 pad 2: /Project Architecture/M.2 Drives/+5V S1 -> /Project Architecture/M.2 Drives/EN
- C74 pad 1: Net-(IC3-PGND2_1) -> gnd
- C74 pad 2: /Project Architecture/M.2 Drives/+5V S1 -> /Project Architecture/M.2 Drives/EN
- C76 pad 1: /Project Architecture/M.2 Drives/+5V S1 -> /Project Architecture/M.2 Drives/EN
- C76 pad 2: Net-(IC3-PGND1_1) -> gnd
- C77 pad 1: /Project Architecture/M.2 Drives/+5V S1 -> /Project Architecture/M.2 Drives/EN
- C77 pad 2: Net-(IC3-PGND1_1) -> gnd
- IC3 pad 1: Net-(IC3-PGND2_1) -> gnd
- IC3 pad 14: /Project Architecture/M.2 Drives/+5V S1 -> /Project Architecture/M.2 Drives/EN
- IC3 pad 15: Net-(IC3-PGND1_1) -> gnd
- IC3 pad 2: /Project Architecture/M.2 Drives/+5V S1 -> /Project Architecture/M.2 Drives/EN
- Module1 pad 88: /Project Architecture/CM5_GPIO/+1V8 -> unconnected-(Module1A-+1.8v_(Output)-Pad88)
- Module1 pad 90: /Project Architecture/CM5_GPIO/+1V8 -> unconnected-(Module1A-+1.8v_(Output)-Pad90)
- U8 pad 2: /Project Architecture/M.2 Drives/gnd{PERST} -> /Project Architecture/M.2 Drives/PERST
