File: Electronics/Project Architecture.kicad_sch (KiCad schematic)
At the start: 5 parts

Commit message: stuff
Other:
- sheet CM5_GPIO: file Section B - TItle B.kicad_sch -> GPIO.kicad_sch
- sheet CM5_High Speed IO: file Section A - Title A.kicad_sch -> High_Speed IO.kicad_sch
- sheet Input: file untitled.kicad_sch -> Input.kicad_sch
- sheet Usb Switch: file USB & Ethernet.kicad_sch -> USB.kicad_sch
- note added: "connecect usb 2"
