File: Electronics/Sata_Drives2.kicad_sch (KiCad schematic)
At the start: 66 parts, among them J20 0877131001, J21 0877131001, Q10 NPN, Q11 PMOS, Q12 NPN, Q13 PMOS, Q14 PMOS, Q15 NPN, Q16 PMOS, Q17 NPN, U11 JMS561, U12 W25X20CLUXIG_TR, Y2 30MHz

Commit message: stuff
Parts:
- added JP6: 3P_JUMPER, Connector_PinHeader_2.54mm:PinHeader_1x03_P2.54mm_Vertical, symbol Jumper:Jumper_3_Bridged12
- added R85: 100K, Resistor_SMD:R_0603_1608Metric, symbol Device:R_Small
Connections:
- net +3V3: now also R85.2
- net gnd: now also JP6.2 (C); no longer U12.3 (~{WP})
- net USB3-1-D_N: now reaches U11.23 (DM)
- net USB3-1-D_P: now reaches U11.24 (DP)
- new net: JP6.1 (A), R85.1, U12.3 (~{WP})
- no-connect marks 16 -> 15
Other:
- moved on the sheet: R72
